File: SC9-STM32F103C8Tx-v2/cs.kicad_pcb (KiCad board)
At the start: 2 copper layers, 25.5 x 21.7 mm, 77 parts, among them J1 SiPM Catode(3) 29.6v, J10 B+, J11 B-, J12 Buzzer, J13 +BAT, J18 I2C-SCL, J19 I2C-SDA, J2 USB_B_Micro, J3 SWDIO, J4 SWCLK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

Commit message: modified:   SC9-STM32F103C8Tx-v2/cs.kicad_pcb 	modified:   SC9-STM32F103C8Tx-v2/cs.kicad_pcb-bak 	modified:   SC9-STM32F103C8Tx-v2/cs.net 	modified:   SC9-STM32F103C8Tx-v2/cs.sch 	modified:   SC9-STM32F103C8Tx-v2/cs.sch-bak
Parts:
- removed D4: JDY-10, My-library:JDY-10
- added J14: RxD, My-library:SMD-CONN, F.Cu at (38.1, 88.6)
- added J15: +BT, My-library:SMD-CONN, F.Cu at (46.1, 77.9)
- added J5: Stat, My-library:SMD-CONN, F.Cu at (36.2, 88.3)
- added J6: TxD, My-library:SMD-CONN, F.Cu at (37.1, 86.7)
