File: SC9-STM32F103C8Tx-v2/cs.sch (KiCad schematic (older format))
At the start: 77 parts, among them J1 SiPM Catode(3) 29.6v, J10 B+, J11 B-, J12 Buzzer, J13 +BAT, J18 I2C-SCL, J19 I2C-SDA, J2 USB_B_Micro, J3 SWDIO, J4 SWCLK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

Commit message: modified:   SC9-STM32F103C8Tx-v2/cs.kicad_pcb 	modified:   SC9-STM32F103C8Tx-v2/cs.kicad_pcb-bak 	modified:   SC9-STM32F103C8Tx-v2/cs.net 	modified:   SC9-STM32F103C8Tx-v2/cs.sch 	modified:   SC9-STM32F103C8Tx-v2/cs.sch-bak
Parts:
- added J14: RxD, My-library:SMD-CONN, symbol cs-rescue:Conn-My_Library
- added J15: +BT, My-library:SMD-CONN, symbol cs-rescue:Conn-My_Library
- added J5: Stat, My-library:SMD-CONN, symbol cs-rescue:Conn-My_Library
- added J6: TxD, My-library:SMD-CONN, symbol cs-rescue:Conn-My_Library
- D4: footprint My-library:JDY-10 -> (none)
Connections:
- net +3V3: now also J15.1 (Pin_1)
- net uart_rxd: now also J14.1 (Pin_1)
- net uart_txd: now also J6.1 (Pin_1)
- net at D4.11 (Stat), U1.26 (PB13): now also J5.1 (Pin_1)
Other:
- moved on the sheet: C1, C10, C11, C12, C13, C14, C15, C16, C17, C18, C19, C2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
