File: SC9-STM32F103C8Tx-v2/cs.sch (KiCad schematic (older format))
At the start: 81 parts, among them J1 SiPM Catode(3) 29.6v, J10 B+, J11 B-, J12 Buzzer, J13 +BAT, J14 RxD, J15 +BT, J18 I2C-SCL, J19 I2C-SDA, J2 USB_B_Micro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

Commit message: изменено:      SC9-STM32F103C8Tx-v2/cs-cache.lib 	изменено:      SC9-STM32F103C8Tx-v2/cs.sch 	изменено:      SC9-STM32F103C8Tx-v2/cs.sch-bak 	изменено:      STM32Code/.cproject 	изменено:      STM32Code/.settings/language.settings.xml 	изменено:      STM32Code/Core/Inc/main.h 	изменено:      STM32Code/Core/Src/main.c 	изменено:      STM32Code/Core/Src/stm32f1xx_hal_msp.c 	изменено:      STM32Code/Core/Src/stm32f1xx_it.c 	изменено:      STM32Code/Release/Core/Src/main.o 	изменено:      STM32Code/Release/Core/Src/main.su 	изменено:      STM32Code/Release/Core/Src/stm32f1xx_hal_msp.o 	изменено:      STM32Code/Release/Core/Src/stm32f1xx_hal_msp.su 	изменено:      STM32Code/Release/Core/Src/stm32f1xx_it.o 	изменено:      STM32Code/Release/SC4-LCD128x32.bin 	изменено:      STM32Code/Release/SC4-LCD128x32.elf 	изменено:      STM32Code/Release/SC4-LCD128x32.list 	изменено:      STM32Code/Release/SC4-LCD128x32.map 	удалено:       STM32Code/SC4-LCD128x32 Debug.launch 	изменено:      STM32Code/SC4-LCD128x32 Release.launch 	изменено:      STM32Code/SC4-LCD128x32.ioc
Parts:
- D4: symbol My_Library:JDY-10 -> cs-rescue:JDY-10-My_Library
Changed lines of the file:
@@
 $EndComp
 $Comp
-L My_Library:JDY-10 D4
+L cs-rescue:JDY-10-My_Library D4
 U 1 1 6021FB35
 P 8250 4950
