File: SC9-STM32F103C8Tx-v3/cs.kicad_pcb (KiCad board)
At the start: 2 copper layers, 25.5 x 21.7 mm, 80 parts, among them J1 SiPM Catode(3) 29.6v, J10 B+, J11 B-, J12 Buzzer, J13 +BAT, J14 RxD, J15 +BT, J18 I2C-SCL, J19 I2C-SDA, J2 USB_B_Micro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

Commit message: изменено:      SC9-STM32F103C8Tx-v3/cs.kicad_pcb 	изменено:      SC9-STM32F103C8Tx-v3/cs.kicad_pcb-bak 	изменено:      SC9-STM32F103C8Tx-v3/cs.net 	изменено:      SC9-STM32F103C8Tx-v3/cs.pdf 	изменено:      SC9-STM32F103C8Tx-v3/cs.sch 	изменено:      SC9-STM32F103C8Tx-v3/cs.sch-bak 	изменено:      SC9-STM32F103C8Tx-v3/fp-info-cache
Parts:
- moved J5 2.59 mm to (33.8, 87.4)
- moved J6 1.57 mm to (35.7, 87.3)
- moved J14 1.43 mm to (37.6, 87.3)
- moved C21 1.07 mm to (34.2, 81.9)
- moved C5 0.50 mm to (27.3, 77.6)
- moved C17 0.47 mm to (30.4, 77.6)
- moved R1 0.27 mm to (30.9, 74.7)
- moved R2 0.26 mm to (27.6, 74.7)
- moved C16 0.22 mm to (29.0, 80.0)
- moved C19 0.08 mm to (44.5, 78.4)
Routing:
- net GND: track 298.9 -> 301.0 mm
- net uart_txd: track 2.20 -> 3.95 mm
- net uart_rxd: track 3.99 -> 2.91 mm
- net +3.3VADC: track 11.1 -> 10.0 mm
