File: SC9-STM32F103C8Tx-v3/cs.sch (KiCad schematic (older format))
At the start: 81 parts, among them J1 SiPM Catode(3) 29.6v, J10 B+, J11 B-, J12 Buzzer, J13 +BAT, J14 RxD, J15 +BT, J18 I2C-SCL, J19 I2C-SDA, J2 USB_B_Micro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

Commit message: изменено:      SC9-STM32F103C8Tx-v3/cs.kicad_pcb 	изменено:      SC9-STM32F103C8Tx-v3/cs.kicad_pcb-bak 	изменено:      SC9-STM32F103C8Tx-v3/cs.net 	изменено:      SC9-STM32F103C8Tx-v3/cs.pdf 	изменено:      SC9-STM32F103C8Tx-v3/cs.sch 	изменено:      SC9-STM32F103C8Tx-v3/cs.sch-bak 	изменено:      SC9-STM32F103C8Tx-v3/fp-info-cache
Parts:
- L2: value 10uH -> LQM21FN100N
- L4, L6: value 47uH -> MLZ2012M470WT000
- U3: value LTC4054ES5-4.2 -> MCP73831T-2ACI/OT
Connections:
- net uart_rxd: no longer names the net of D4.15 (TxD), J14.1 (Pin_1), U1.31 (PA10)
- net uart_txd: no longer names the net of D4.14 (RxD), J6.1 (Pin_1), U1.30 (PA9)
Other:
- moved on the sheet: C1, C10, C11, C12, C13, C14, C15, C16, C17, C18, C19, C2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
