File: SC-STM32L412K8/SC-STM32L412K8.sch (KiCad schematic (older format))
At the start: 59 parts, among them J1 usb, J2 +29.6, J3 TxD, J4 RxD, J5 SWDIO, J6 SWCLK, J7 +BAT, J8 SiPM-, J9 BT Status, Q1 IRLML5203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

Commit message: SC-STM32L412K8/SC-STM32L412K8-rescue.dcm 	SC-STM32L412K8/SC-STM32L412K8-rescue.lib 	SC-STM32L412K8/sym-lib-table
Parts:
- D6: symbol My_Library:STM32L412K8 -> SC-STM32L412K8-rescue:STM32L412K8-My_Library
- J2, J3, J4, J5, J6, J7, J8, J9: symbol My_Library:Conn -> SC-STM32L412K8-rescue:Conn-My_Library
- U4: symbol My_Library:LMV7239M5 -> SC-STM32L412K8-rescue:LMV7239M5-My_Library
Changed lines of the file:
@@
 $EndDescr
 $Comp
-L My_Library:STM32L412K8 D6
+L SC-STM32L412K8-rescue:STM32L412K8-My_Library D6
 U 1 1 60361EE9
 P 7350 4450
@@
 $EndComp
 $Comp
-L My_Library:Conn J5
+L SC-STM32L412K8-rescue:Conn-My_Library J5
 U 1 1 603AE044
 P 6750 5250
@@
 $EndComp
 $Comp
-L My_Library:Conn J6
+L SC-STM32L412K8-rescue:Conn-My_Library J6
 U 1 1 603AE9C5
 P 6750 5350
@@
 $EndComp
 $Comp
-L My_Library:Conn J3
+L SC-STM32L412K8-rescue:Conn-My_Library J3
 U 1 1 603B523F
 P 6750 4850
@@
 $EndComp
 $Comp
-L My_Library:Conn J4
+L SC-STM32L412K8-rescue:Conn-My_Library J4
 U 1 1 603B58EC
 P 6750 4950
@@
 Connection ~ 3850 1450
 $Comp
-L My_Library:Conn J2
+L SC-STM32L412K8-rescue:Conn-My_Library J2
 U 1 1 604E175B
 P 6150 1450
@@
 Connection ~ 7950 3750
 $Comp
-L My_Library:Conn J7
+L SC-STM32L412K8-rescue:Conn-My_Library J7
 U 1 1 60622710
 P 5200 3700
@@
 Connection ~ 5200 3600
 $Comp
-L My_Library:Conn J8
+L SC-STM32L412K8-rescue:Conn-My_Library J8
 U 1 1 606AB650
 P 5250 5050
@@
 $EndComp
 $Comp
-L My_Library:Conn J9
+L SC-STM32L412K8-rescue:Conn-My_Library J9
 U 1 1 6072E770
 P 6750 5450
@@
 	5350 3600 5350 2900
 $Comp
-L My_Library:LMV7239M5 U4
+L SC-STM32L412K8-rescue:LMV7239M5-My_Library U4
 U 1 1 6056F677
 P 6200 5050

Commit message: modified:   SC-STM32L412K8/SC-STM32L412K8-cache.lib 	modified:   SC-STM32L412K8/SC-STM32L412K8.kicad_pcb 	modified:   SC-STM32L412K8/SC-STM32L412K8.kicad_pcb-bak 	modified:   SC-STM32L412K8/SC-STM32L412K8.net 	modified:   SC-STM32L412K8/SC-STM32L412K8.sch 	modified:   SC-STM32L412K8/SC-STM32L412K8.sch-bak
Parts:
- added J?: PWM, My-library:SMD-CONN, symbol SC-STM32L412K8-rescue:Conn-My_Library-SC-STM32L412K8-rescue
- D6: symbol SC-STM32L412K8-rescue:STM32L412K8-My_Library -> SC-STM32L412K8-rescue:STM32L412K8-My_Library-SC-STM32L412K8-rescue
- J2, J3, J4, J5, J6, J7, J8, J9: symbol SC-STM32L412K8-rescue:Conn-My_Library -> SC-STM32L412K8-rescue:Conn-My_Library-SC-STM32L412K8-rescue
- U4: symbol SC-STM32L412K8-rescue:LMV7239M5-My_Library -> SC-STM32L412K8-rescue:LMV7239M5-My_Library-SC-STM32L412K8-rescue
Connections:
- net at D6.22 (PA12): now also J?.1 (Pin_1)
Changed lines of the file:
@@
 $EndDescr
 $Comp
-L SC-STM32L412K8-rescue:STM32L412K8-My_Library D6
+L SC-STM32L412K8-rescue:STM32L412K8-My_Library-SC-STM32L412K8-rescue D6
 U 1 1 60361EE9
 P 7350 4450
@@
 $EndComp
 $Comp
-L SC-STM32L412K8-rescue:Conn-My_Library J5
+L SC-STM32L412K8-rescue:Conn-My_Library-SC-STM32L412K8-rescue J5
 U 1 1 603AE044
 P 6750 5250
@@
 $EndComp
 $Comp
-L SC-STM32L412K8-rescue:Conn-My_Library J6
+L SC-STM32L412K8-rescue:Conn-My_Library-SC-STM32L412K8-rescue J6
 U 1 1 603AE9C5
 P 6750 5350
@@
 $EndComp
 $Comp
-L SC-STM32L412K8-rescue:Conn-My_Library J3
+L SC-STM32L412K8-rescue:Conn-My_Library-SC-STM32L412K8-rescue J3
 U 1 1 603B523F
 P 6750 4850
@@
 $EndComp
 $Comp
-L SC-STM32L412K8-rescue:Conn-My_Library J4
+L SC-STM32L412K8-rescue:Conn-My_Library-SC-STM32L412K8-rescue J4
 U 1 1 603B58EC
 P 6750 4950
@@
 Connection ~ 3850 1450
 $Comp
-L SC-STM32L412K8-rescue:Conn-My_Library J2
+L SC-STM32L412K8-rescue:Conn-My_Library-SC-STM32L412K8-rescue J2
 U 1 1 604E175B
 P 6150 1450
@@
 Connection ~ 7950 3750
 $Comp
-L SC-STM32L412K8-rescue:Conn-My_Library J7
+L SC-STM32L412K8-rescue:Conn-My_Library-SC-STM32L412K8-rescue J7
 U 1 1 60622710
 P 5200 3700
@@
 Connection ~ 5200 3600
 $Comp
-L SC-STM32L412K8-rescue:Conn-My_Library J8
+L SC-STM32L412K8-rescue:Conn-My_Library-SC-STM32L412K8-rescue J8
 U 1 1 606AB650
 P 5250 5050
@@
 $EndComp
 $Comp
-L SC-STM32L412K8-rescue:Conn-My_Library J9
+L SC-STM32L412K8-rescue:Conn-My_Library-SC-STM32L412K8-rescue J9
 U 1 1 6072E770
 P 6750 5450
@@
 	5350 3600 5350 2900
 $Comp
-L SC-STM32L412K8-rescue:LMV7239M5-My_Library U4
+L SC-STM32L412K8-rescue:LMV7239M5-My_Library-SC-STM32L412K8-rescue U4
 U 1 1 6056F677
 P 6200 5050
@@
 Wire Wire Line
 	6300 4500 6150 4500
+$Comp
+L SC-STM32L412K8-rescue:Conn-My_Library-SC-STM32L412K8-rescue J?
+U 1 1 604B8416
+P 6750 5150
+F 0 "J?" H 6692 4925 50  0001 C CNN
+F 1 "PWM" H 6900 5150 50  0000 C CNN
+F 2 "My-library:SMD-CONN" H 6750 5150 50  0001 C CNN
+F 3 "~" H 6750 5150 50  0001 C CNN
+	1    6750 5150
+	-1   0    0    1
+$EndComp
 $EndSCHEMATC

Commit message: modified:   SC-STM32L412K8/SC-STM32L412K8.kicad_pcb 	modified:   SC-STM32L412K8/SC-STM32L412K8.kicad_pcb-bak 	modified:   SC-STM32L412K8/SC-STM32L412K8.sch 	modified:   SC-STM32L412K8/SC-STM32L412K8.sch-bak
Parts:
- gave numbers to parts that had none: 1
Other:
- moved on the sheet: C6, R2, R7, R8, R9
Changed lines of the file:
@@
 L Device:R R7
 U 1 1 6036B072
-P 5550 4700
-F 0 "R7" H 5350 4800 50  0000 L CNN
-F 1 "100k" H 5300 4700 50  0000 L CNN
-F 2 "Resistor_SMD:R_0603_1608Metric" V 5480 4700 50  0001 C CNN
-F 3 "~" H 5550 4700 50  0001 C CNN
-	1    5550 4700
+P 5500 4700
+F 0 "R7" H 5500 5100 50  0000 L CNN
+F 1 "100k" H 5450 5000 50  0000 L CNN
+F 2 "Resistor_SMD:R_0603_1608Metric" V 5430 4700 50  0001 C CNN
+F 3 "~" H 5500 4700 50  0001 C CNN
+	1    5500 4700
 	1    0    0    -1
 $EndComp
@@
 L Device:R R8
 U 1 1 6036B7B6
-P 5550 5000
-F 0 "R8" H 5620 5046 50  0000 L CNN
-F 1 "220" H 5620 4955 50  0000 L CNN
-F 2 "Resistor_SMD:R_0603_1608Metric" V 5480 5000 50  0001 C CNN
-F 3 "~" H 5550 5000 50  0001 C CNN
-	1    5550 5000
+P 5500 5000
+F 0 "R8" H 5570 5046 50  0000 L CNN
+F 1 "220" H 5570 4955 50  0000 L CNN
+F 2 "Resistor_SMD:R_0603_1608Metric" V 5430 5000 50  0001 C CNN
+F 3 "~" H 5500 5000 50  0001 C CNN
+	1    5500 5000
 	1    0    0    -1
 $EndComp
@@
 L Device:R R9
 U 1 1 6036BC49
-P 5550 5350
-F 0 "R9" H 5620 5396 50  0000 L CNN
-F 1 "12k" H 5620 5305 50  0000 L CNN
-F 2 "Resistor_SMD:R_0603_1608Metric" V 5480 5350 50  0001 C CNN
-F 3 "~" H 5550 5350 50  0001 C CNN
-	1    5550 5350
+P 5500 5350
+F 0 "R9" H 5570 5396 50  0000 L CNN
+F 1 "12k" H 5570 5305 50  0000 L CNN
+F 2 "Resistor_SMD:R_0603_1608Metric" V 5430 5350 50  0001 C CNN
+F 3 "~" H 5500 5350 50  0001 C CNN
+	1    5500 5350
 	1    0    0    -1
 $EndComp
@@
 L Device:C C6
 U 1 1 6036D36F
-P 5400 5150
-F 0 "C6" V 5148 5150 50  0000 C CNN
-F 1 "470pF" V 5239 5150 50  0000 C CNN
-F 2 "Capacitor_SMD:C_0603_1608Metric" H 5438 5000 50  0001 C CNN
-F 3 "~" H 5400 5150 50  0001 C CNN
-	1    5400 5150
+P 5350 5150
+F 0 "C6" V 5098 5150 50  0000 C CNN
+F 1 "470pF" V 5189 5150 50  0000 C CNN
+F 2 "Capacitor_SMD:C_0603_1608Metric" H 5388 5000 50  0001 C CNN
+F 3 "~" H 5350 5150 50  0001 C CNN
+	1    5350 5150
 	0    1    1    0
 $EndComp
@@
 L Device:R R2
 U 1 1 6036DAFE
-P 5250 5350
-F 0 "R2" H 5320 5396 50  0000 L CNN
-F 1 "2.2k" H 5320 5305 50  0000 L CNN
-F 2 "Resistor_SMD:R_0603_1608Metric" V 5180 5350 50  0001 C CNN
-F 3 "~" H 5250 5350 50  0001 C CNN
-	1    5250 5350
+P 5200 5350
+F 0 "R2" H 5270 5396 50  0000 L CNN
+F 1 "2.2k" H 5270 5305 50  0000 L CNN
+F 2 "Resistor_SMD:R_0603_1608Metric" V 5130 5350 50  0001 C CNN
+F 3 "~" H 5200 5350 50  0001 C CNN
+	1    5200 5350
 	1    0    0    -1
 $EndComp
@@
 Text GLabel 7950 4300 2    50   Input ~ 0
 AIn
-Text GLabel 5150 5150 0    50   Input ~ 0
+Text GLabel 5100 5150 0    50   Input ~ 0
 AIn
 $Comp
@@
 L SC-STM32L412K8-rescue:Conn-My_Library-SC-STM32L412K8-rescue J8
 U 1 1 606AB650
-P 5250 5050
-F 0 "J8" H 5192 4825 50  0001 C CNN
-F 1 "SiPM-" V 5250 5200 50  0000 C CNN
-F 2 "My-library:SMD-CONN" H 5250 5050 50  0001 C CNN
-F 3 "~" H 5250 5050 50  0001 C CNN
-	1    5250 5050
+P 5200 5050
+F 0 "J8" H 5142 4825 50  0001 C CNN
+F 1 "SiPM-" V 5200 5200 50  0000 C CNN
+F 2 "My-library:SMD-CONN" H 5200 5050 50  0001 C CNN
+F 3 "~" H 5200 5050 50  0001 C CNN
+	1    5200 5050
 	0    -1   -1   0
 $EndComp
@@
 Wire Wire Line
 	7500 3400 7950 3400
-Connection ~ 5550 4850
-Wire Wire Line
-	5550 4550 5550 4500
-Wire Wire Line
-	5550 4500 6150 4500
 Wire Wire Line
 	6150 5300 6150 5500
@@
 	6150 5500 5850 5500
 Connection ~ 6150 5500
-Connection ~ 5550 5500
-Wire Wire Line
-	5550 5500 5250 5500
 Connection ~ 5850 5500
-Wire Wire Line
-	5850 5500 5550 5500
-Wire Wire Line
-	5150 5150 5250 5150
-Wire Wire Line
-	5250 5150 5250 5200
-Connection ~ 5250 5150
-Wire Wire Line
-	5550 5200 5550 5150
-Wire Wire Line
-	5550 5150 5950 5150
-Connection ~ 5550 5150
 Wire Wire Line
 	5850 5200 5850 4950
@@
 	5200 4900 4750 4900
 Wire Wire Line
-	5150 4500 5550 4500
-Connection ~ 5550 4500
-Wire Wire Line
-	4250 5500 5250 5500
-Connection ~ 5250 5500
+	5150 4500 5500 4500
+Wire Wire Line
+	4250 5500 5200 5500
 Wire Wire Line
 	6550 5050 6850 5050
@@
 	6300 4500 6150 4500
 $Comp
-L SC-STM32L412K8-rescue:Conn-My_Library-SC-STM32L412K8-rescue J?
+L SC-STM32L412K8-rescue:Conn-My_Library-SC-STM32L412K8-rescue J10
 U 1 1 604B8416
 P 6750 5150
-F 0 "J?" H 6692 4925 50  0001 C CNN
+F 0 "J10" H 6692 4925 50  0001 C CNN
 F 1 "PWM" H 6900 5150 50  0000 C CNN
 F 2 "My-library:SMD-CONN" H 6750 5150 50  0001 C CNN
@@
 	-1   0    0    1
 $EndComp
+Connection ~ 5200 5150
+Wire Wire Line
+	5200 5150 5250 5150
+Connection ~ 5200 5500
+Connection ~ 5500 5500
+Wire Wire Line
+	5550 4850 5500 4850
+Wire Wire Line
+	5500 5500 5850 5500
+Wire Wire Line
+	5200 5500 5500 5500
+Connection ~ 5500 4850
+Wire Wire Line
+	5500 4550 5500 4500
+Connection ~ 5500 4500
+Wire Wire Line
+	5500 4500 6150 4500
+Wire Wire Line
+	5100 5150 5200 5150
+Wire Wire Line
+	5200 5150 5200 5200
+Wire Wire Line
+	5500 5200 5500 5150
+Connection ~ 5500 5150
+Wire Wire Line
+	5500 5150 5950 5150
 $EndSCHEMATC

Commit message: modified:   SC-STM32L412K8/SC-STM32L412K8-cache.lib 	modified:   SC-STM32L412K8/SC-STM32L412K8.kicad_pcb 	modified:   SC-STM32L412K8/SC-STM32L412K8.kicad_pcb-bak 	modified:   SC-STM32L412K8/SC-STM32L412K8.net 	modified:   SC-STM32L412K8/SC-STM32L412K8.sch 	modified:   SC-STM32L412K8/SC-STM32L412K8.sch-bak
Parts:
- added BZ1: Buzzer, My-library:BuzerSMD, symbol Device:Buzzer
- added J11: Vibro, My-library:SMD-CONN, symbol SC-STM32L412K8-rescue:Conn-My_Library-SC-STM32L412K8-rescue
- added J12: +3v, My-library:SMD-CONN, symbol SC-STM32L412K8-rescue:Conn-My_Library-SC-STM32L412K8-rescue
- added Q2, Q3: KT235, Package_TO_SOT_SMD:SOT-23, symbol Device:Q_NPN_BEC
- added R15, R16: 4.7k, Resistor_SMD:R_0603_1608Metric, symbol Device:R
Connections:
- net +BATT: now also BZ1.1 (-)
- net GND: now also Q2.2 (E), Q3.2 (E)
- net at C16.1, C17.1, C19.1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: now also J12.1 (Pin_1)
- net Buzer: now reaches D6.10 (PA4)
- net Buzer: now also R15.2
- net Vibro: now reaches D6.7 (PA1)
- net Vibro: now also R16.2
- new net: Q2.1 (B), R15.1
- new net: BZ1.2 (+), Q2.3 (C)
- new net: Q3.1 (B), R16.1
- new net: J11.1 (Pin_1), Q3.3 (C)
Other:
- moved on the sheet: C16, C17

Commit message: modified:   SC-STM32L412K8/SC-STM32L412K8.kicad_pcb 	modified:   SC-STM32L412K8/SC-STM32L412K8.kicad_pcb-bak 	modified:   SC-STM32L412K8/SC-STM32L412K8.net 	modified:   SC-STM32L412K8/SC-STM32L412K8.sch 	modified:   SC-STM32L412K8/SC-STM32L412K8.sch-bak 	modified:   STM32Code/.settings/language.settings.xml 	modified:   STM32Code/Core/Src/main.c 	modified:   STM32Code/Release/Core/Src/main.o 	modified:   STM32Code/Release/Core/Src/main.su 	modified:   STM32Code/Release/SC4-LCD128x32.bin 	modified:   STM32Code/Release/SC4-LCD128x32.elf 	modified:   STM32Code/Release/SC4-LCD128x32.list 	modified:   STM32Code/Release/SC4-LCD128x32.map 	modified:   STM32Code/Release/makefile
Parts:
- added J13: +vibro, My-library:SMD-CONN, symbol SC-STM32L412K8-rescue:Conn-My_Library-SC-STM32L412K8-rescue
- added R17, R18: X, Resistor_SMD:R_0603_1608Metric, symbol Device:R
- J2: value +29.6 -> +29.6 SiPM
Connections:
- net +BATT: now also J13.1 (Pin_1)
- net GND: now also R18.1
- net at C16.1, C17.1, C19.1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: now also R17.2
- net tm: now reaches D6.14 (PB0)
- net tm: now also R17.1, R18.2
Other:
- moved on the sheet: BZ1, Q2, Q3, R15, R16
Changed lines of the file:
@@
 U 1 1 6037B2E7
 P 7500 3550
-F 0 "L4" H 7553 3596 50  0000 L CNN
-F 1 "47uH" H 7550 3500 50  0000 L CNN
+F 0 "L4" H 7500 3850 50  0000 L CNN
+F 1 "47uH" H 7500 3750 50  0000 L CNN
 F 2 "Inductor_SMD:L_0805_2012Metric" H 7500 3550 50  0001 C CNN
 F 3 "~" H 7500 3550 50  0001 C CNN
@@
 U 1 1 6037FBDB
 P 7700 3750
-F 0 "C18" V 7500 3900 50  0000 C CNN
-F 1 "22uF" V 7600 3950 50  0000 C CNN
+F 0 "C18" V 7450 3750 50  0000 C CNN
+F 1 "22uF" V 7550 3750 50  0000 C CNN
 F 2 "Capacitor_SMD:C_0805_2012Metric" H 7738 3600 50  0001 C CNN
 F 3 "~" H 7700 3750 50  0001 C CNN
@@
 U 1 1 6039B0E7
 P 7200 3550
-F 0 "C17" H 7200 3900 50  0000 L CNN
-F 1 "22uF" H 7200 3800 50  0000 L CNN
+F 0 "C17" H 7200 3850 50  0000 L CNN
+F 1 "22uF" H 7200 3750 50  0000 L CNN
 F 2 "Capacitor_SMD:C_0805_2012Metric" H 7238 3400 50  0001 C CNN
 F 3 "~" H 7200 3550 50  0001 C CNN
@@
 U 1 1 603AB7C1
 P 7000 3550
-F 0 "C16" H 6950 3900 50  0000 L CNN
-F 1 "22uF" H 6950 3800 50  0000 L CNN
+F 0 "C16" H 6950 3850 50  0000 L CNN
+F 1 "22uF" H 6950 3750 50  0000 L CNN
 F 2 "Capacitor_SMD:C_0805_2012Metric" H 7038 3400 50  0001 C CNN
 F 3 "~" H 7000 3550 50  0001 C CNN
@@
 P 6150 1450
 F 0 "J2" H 6092 1225 50  0001 C CNN
-F 1 "+29.6" H 6050 1600 50  0000 C CNN
+F 1 "+29.6 SiPM" H 6050 1600 50  0000 C CNN
 F 2 "My-library:SMD-CONN" H 6150 1450 50  0001 C CNN
 F 3 "~" H 6150 1450 50  0001 C CNN
@@
 U 1 1 604E38DC
 P 6050 3150
-F 0 "SW1" H 6050 3435 50  0000 C CNN
-F 1 "power" H 6050 3344 50  0000 C CNN
+F 0 "SW1" H 6000 3300 50  0000 C CNN
+F 1 "power" H 6000 3000 50  0000 C CNN
 F 2 "My-library:MySwithc" H 6050 3150 50  0001 C CNN
 F 3 "" H 6050 3150 50  0001 C CNN
@@
 L Device:Q_NPN_BEC Q2
 U 1 1 604F8B65
-P 7250 2200
-F 0 "Q2" H 7441 2246 50  0000 L CNN
-F 1 "KT235" H 7441 2155 50  0000 L CNN
-F 2 "Package_TO_SOT_SMD:SOT-23" H 7450 2300 50  0001 C CNN
-F 3 "~" H 7250 2200 50  0001 C CNN
-	1    7250 2200
+P 7050 2200
+F 0 "Q2" H 7241 2246 50  0000 L CNN
+F 1 "KT235" H 7241 2155 50  0000 L CNN
+F 2 "Package_TO_SOT_SMD:SOT-23" H 7250 2300 50  0001 C CNN
+F 3 "~" H 7050 2200 50  0001 C CNN
+	1    7050 2200
 	1    0    0    -1
 $EndComp
@@
 L Device:Q_NPN_BEC Q3
 U 1 1 604F994F
-P 7250 1400
-F 0 "Q3" H 6800 1250 50  0000 L CNN
-F 1 "KT235" H 7000 1250 50  0000 L CNN
-F 2 "Package_TO_SOT_SMD:SOT-23" H 7450 1500 50  0001 C CNN
-F 3 "~" H 7250 1400 50  0001 C CNN
-	1    7250 1400
+P 7050 1400
+F 0 "Q3" H 6600 1250 50  0000 L CNN
+F 1 "KT235" H 6800 1250 50  0000 L CNN
+F 2 "Package_TO_SOT_SMD:SOT-23" H 7250 1500 50  0001 C CNN
+F 3 "~" H 7050 1400 50  0001 C CNN
+	1    7050 1400
 	1    0    0    -1
 $EndComp
@@
 L Device:R R15
 U 1 1 604FA546
-P 6900 2200
-F 0 "R15" V 6700 2150 50  0000 C CNN
-F 1 "4.7k" V 6800 2150 50  0000 C CNN
-F 2 "Resistor_SMD:R_0603_1608Metric" V 6830 2200 50  0001 C CNN
-F 3 "~" H 6900 2200 50  0001 C CNN
-	1    6900 2200
+P 6700 2200
+F 0 "R15" V 6500 2150 50  0000 C CNN
+F 1 "4.7k" V 6600 2150 50  0000 C CNN
+F 2 "Resistor_SMD:R_0603_1608Metric" V 6630 2200 50  0001 C CNN
+F 3 "~" H 6700 2200 50  0001 C CNN
+	1    6700 2200
 	0    1    1    0
 $EndComp
@@
 L Device:R R16
 U 1 1 604FB12B
-P 6900 1400
-F 0 "R16" V 6700 1600 50  0000 C CNN
-F 1 "4.7k" V 6800 1600 50  0000 C CNN
-F 2 "Resistor_SMD:R_0603_1608Metric" V 6830 1400 50  0001 C CNN
-F 3 "~" H 6900 1400 50  0001 C CNN
-	1    6900 1400
+P 6700 1400
+F 0 "R16" V 6500 1600 50  0000 C CNN
+F 1 "4.7k" V 6600 1600 50  0000 C CNN
+F 2 "Resistor_SMD:R_0603_1608Metric" V 6630 1400 50  0001 C CNN
+F 3 "~" H 6700 1400 50  0001 C CNN
+	1    6700 1400
 	0    1    1    0
 $EndComp
@@
 L power:GND #PWR0101
 U 1 1 604FBD4D
-P 7350 2400
-F 0 "#PWR0101" H 7350 2150 50  0001 C CNN
-F 1 "GND" H 7355 2227 50  0001 C CNN
-F 2 "" H 7350 2400 50  0001 C CNN
-F 3 "" H 7350 2400 50  0001 C CNN
-	1    7350 2400
+P 7150 2400
+F 0 "#PWR0101" H 7150 2150 50  0001 C CNN
+F 1 "GND" H 7155 2227 50  0001 C CNN
+F 2 "" H 7150 2400 50  0001 C CNN
+F 3 "" H 7150 2400 50  0001 C CNN
+	1    7150 2400
 	1    0    0    -1
 $EndComp
@@
 L power:GND #PWR0102
 U 1 1 604FC90E
-P 7350 1600
-F 0 "#PWR0102" H 7350 1350 50  0001 C CNN
-F 1 "GND" H 7355 1427 50  0001 C CNN
-F 2 "" H 7350 1600 50  0001 C CNN
-F 3 "" H 7350 1600 50  0001 C CNN
-	1    7350 1600
+P 7150 1600
+F 0 "#PWR0102" H 7150 1350 50  0001 C CNN
+F 1 "GND" H 7155 1427 50  0001 C CNN
+F 2 "" H 7150 1600 50  0001 C CNN
+F 3 "" H 7150 1600 50  0001 C CNN
+	1    7150 1600
 	1    0    0    -1
 $EndComp
@@
 L Device:Buzzer BZ1
 U 1 1 604FDD84
-P 7450 1900
-F 0 "BZ1" H 7602 1929 50  0000 L CNN
-F 1 "Buzzer" H 7602 1838 50  0000 L CNN
-F 2 "My-library:BuzerSMD" V 7425 2000 50  0001 C CNN
-F 3 "~" V 7425 2000 50  0001 C CNN
-	1    7450 1900
+P 7250 1900
+F 0 "BZ1" H 7402 1929 50  0000 L CNN
+F 1 "Buzzer" H 7402 1838 50  0000 L CNN
+F 2 "My-library:BuzerSMD" V 7225 2000 50  0001 C CNN
+F 3 "~" V 7225 2000 50  0001 C CNN
+	1    7250 1900
 	1    0    0    -1
 $EndComp
@@
 L power:+BATT #PWR0103
 U 1 1 60504BD6
-P 7350 1800
-F 0 "#PWR0103" H 7350 1650 50  0001 C CNN
-F 1 "+BATT" V 7350 2050 50  0000 C CNN
-F 2 "" H 7350 1800 50  0001 C CNN
-F 3 "" H 7350 1800 50  0001 C CNN
-	1    7350 1800
+P 7150 1800
+F 0 "#PWR0103" H 7150 1650 50  0001 C CNN
+F 1 "+BATT" V 7150 2050 50  0000 C CNN
+F 2 "" H 7150 1800 50  0001 C CNN
+F 3 "" H 7150 1800 50  0001 C CNN
+	1    7150 1800
 	0    -1   -1   0
 $EndComp
@@
 L SC-STM32L412K8-rescue:Conn-My_Library-SC-STM32L412K8-rescue J11
 U 1 1 605058F1
-P 7450 1200
-F 0 "J11" H 7392 975 50  0001 C CNN
-F 1 "Vibro" H 7350 1350 50  0000 C CNN
-F 2 "My-library:SMD-CONN" H 7450 1200 50  0001 C CNN
-F 3 "~" H 7450 1200 50  0001 C CNN
-	1    7450 1200
+P 7250 1200
+F 0 "J11" H 7192 975 50  0001 C CNN
+F 1 "Vibro" H 7150 1350 50  0000 C CNN
+F 2 "My-library:SMD-CONN" H 7250 1200 50  0001 C CNN
+F 3 "~" H 7250 1200 50  0001 C CNN
+	1    7250 1200
 	1    0    0    -1
 $EndComp
@@
 $EndComp
 Connection ~ 7950 2800
-Text GLabel 6750 1400 0    50   Input ~ 0
+Text GLabel 6550 1400 0    50   Input ~ 0
 Vibro
 Text GLabel 6850 4050 0    50   Input ~ 0
 Vibro
-Text GLabel 6750 2200 0    50   Input ~ 0
+Text GLabel 6550 2200 0    50   Input ~ 0
 Buzer
 Text GLabel 6850 4350 0    50   Input ~ 0
 Buzer
+$Comp
+L SC-STM32L412K8-rescue:Conn-My_Library-SC-STM32L412K8-rescue J13
+U 1 1 6052B033
+P 6450 3250
+F 0 "J13" H 6392 3025 50  0001 C CNN
+F 1 "+vibro" H 6450 3150 50  0000 C CNN
+F 2 "My-library:SMD-CONN" H 6450 3250 50  0001 C CNN
+F 3 "~" H 6450 3250 50  0001 C CNN
+	1    6450 3250
+	1    0    0    -1
+$EndComp
+Connection ~ 6350 3250
+$Comp
+L Device:R R17
+U 1 1 6056FB73
+P 8100 2950
+F 0 "R17" H 7950 2950 50  0000 C CNN
+F 1 "X" H 7950 2850 50  0000 C CNN
+F 2 "Resistor_SMD:R_0603_1608Metric" V 8030 2950 50  0001 C CNN
+F 3 "~" H 8100 2950 50  0001 C CNN
+	1    8100 2950
+	-1   0    0    1
+$EndComp
+$Comp
+L Device:R R18
+U 1 1 60570A8B
+P 8100 3250
+F 0 "R18" H 7950 3350 50  0000 C CNN
+F 1 "X" H 7950 3250 50  0000 C CNN
+F 2 "Resistor_SMD:R_0603_1608Metric" V 8030 3250 50  0001 C CNN
+F 3 "~" H 8100 3250 50  0001 C CNN
+	1    8100 3250
+	-1   0    0    1
+$EndComp
+$Comp
+L power:GND #PWR05
+U 1 1 6057F52E
+P 8100 3400
+F 0 "#PWR05" H 8100 3150 50  0001 C CNN
+F 1 "GND" H 8105 3227 50  0001 C CNN
+F 2 "" H 8100 3400 50  0001 C CNN
+F 3 "" H 8100 3400 50  0001 C CNN
+	1    8100 3400
+	1    0    0    -1
+$EndComp
+Text GLabel 8300 3100 2    50   Input ~ 0
+tm
+Wire Wire Line
+	8100 3100 8300 3100
+Connection ~ 8100 3100
+Wire Wire Line
+	7950 2800 8100 2800
+Text GLabel 7950 4200 2    50   Input ~ 0
+tm
 $EndSCHEMATC

Commit message: modified:   SC-STM32L412K8/SC-STM32L412K8.kicad_pcb 	modified:   SC-STM32L412K8/SC-STM32L412K8.kicad_pcb-bak 	modified:   SC-STM32L412K8/SC-STM32L412K8.net 	modified:   SC-STM32L412K8/SC-STM32L412K8.sch 	modified:   SC-STM32L412K8/SC-STM32L412K8.sch-bak
Parts:
- added R19, R20: X, Resistor_SMD:R_0603_1608Metric, symbol Device:R
Connections:
- net +BATT: now also R19.2
- net GND: now also R20.1
- net tm: now also D6.12 (PA6); no longer D6.14 (PB0)
- net bl: now reaches D6.13 (PA7)
- net bl: now also R19.1, R20.2
Changed lines of the file:
@@
 Wire Wire Line
 	7950 2800 8100 2800
-Text GLabel 7950 4200 2    50   Input ~ 0
+Text GLabel 6850 4550 0    50   Input ~ 0
 tm
+$Comp
+L Device:R R19
+U 1 1 60539C8E
+P 7750 1650
+F 0 "R19" H 7600 1650 50  0000 C CNN
+F 1 "X" H 7600 1550 50  0000 C CNN
+F 2 "Resistor_SMD:R_0603_1608Metric" V 7680 1650 50  0001 C CNN
+F 3 "~" H 7750 1650 50  0001 C CNN
+	1    7750 1650
+	-1   0    0    1
+$EndComp
+$Comp
+L Device:R R20
+U 1 1 6053A8EC
+P 7750 1950
+F 0 "R20" H 7600 2050 50  0000 C CNN
+F 1 "X" H 7600 1950 50  0000 C CNN
+F 2 "Resistor_SMD:R_0603_1608Metric" V 7680 1950 50  0001 C CNN
+F 3 "~" H 7750 1950 50  0001 C CNN
+	1    7750 1950
+	-1   0    0    1
+$EndComp
+$Comp
+L power:GND #PWR0104
+U 1 1 6053B5D1
+P 7750 2100
+F 0 "#PWR0104" H 7750 1850 50  0001 C CNN
+F 1 "GND" H 7755 1927 50  0001 C CNN
+F 2 "" H 7750 2100 50  0001 C CNN
+F 3 "" H 7750 2100 50  0001 C CNN
+	1    7750 2100
+	1    0    0    -1
+$EndComp
+$Comp
+L power:+BATT #PWR0105
+U 1 1 605487AC
+P 7750 1500
+F 0 "#PWR0105" H 7750 1350 50  0001 C CNN
+F 1 "+BATT" H 7850 1650 50  0000 C CNN
+F 2 "" H 7750 1500 50  0001 C CNN
+F 3 "" H 7750 1500 50  0001 C CNN
+	1    7750 1500
+	1    0    0    -1
+$EndComp
+Text GLabel 7950 1800 2    50   Input ~ 0
+bl
+Wire Wire Line
+	7750 1800 7950 1800
+Connection ~ 7750 1800
+Text GLabel 6850 4650 0    50   Input ~ 0
+bl
 $EndSCHEMATC
