File: SC-STM32L412K8/SC-STM32L412K8.sch (KiCad schematic (older format))
At the start: 72 parts, among them J1 usb, J10 PWM, J11 Vibro, J12 +3v, J13 +vibro, J2 +29.6 SiPM, J3 TxD, J4 RxD, J5 SWDIO, J6 SWCLK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

Commit message: изменено:      SC-STM32L412K8/SC-STM32L412K8-cache.lib 	изменено:      SC-STM32L412K8/SC-STM32L412K8.kicad_pcb 	изменено:      SC-STM32L412K8/SC-STM32L412K8.kicad_pcb-bak 	изменено:      SC-STM32L412K8/SC-STM32L412K8.sch 	изменено:      SC-STM32L412K8/SC-STM32L412K8.sch-bak 	SC-STM32L412K8/SC-STM32L412K8-rescue.dcm 	SC-STM32L412K8/SC-STM32L412K8-rescue.lib
Parts:
- D6: symbol SC-STM32L412K8-rescue:STM32L412K8-My_Library-SC-STM32L412K8-rescue -> SC-STM32L412K8-rescue:STM32L412K8-My_Library-SC-STM32L412K8-rescue-SC-STM32L412K8-rescue
- J10, J11, J12, J13, J2, J3, J4, J5, J6, J7, J8, J9: symbol SC-STM32L412K8-rescue:Conn-My_Library-SC-STM32L412K8-rescue -> SC-STM32L412K8-rescue:Conn-My_Library-SC-STM32L412K8-rescue-SC-STM32L412K8-rescue
- U4: symbol SC-STM32L412K8-rescue:LMV7239M5-My_Library-SC-STM32L412K8-rescue -> SC-STM32L412K8-rescue:LMV7239M5-My_Library-SC-STM32L412K8-rescue-SC-STM32L412K8-rescue
Changed lines of the file:
@@
 $EndDescr
 $Comp
-L SC-STM32L412K8-rescue:STM32L412K8-My_Library-SC-STM32L412K8-rescue D6
+L SC-STM32L412K8-rescue:STM32L412K8-My_Library-SC-STM32L412K8-rescue-SC-STM32L412K8-rescue D6
 U 1 1 60361EE9
 P 7350 4450
@@
 $EndComp
 $Comp
-L SC-STM32L412K8-rescue:Conn-My_Library-SC-STM32L412K8-rescue J5
+L SC-STM32L412K8-rescue:Conn-My_Library-SC-STM32L412K8-rescue-SC-STM32L412K8-rescue J5
 U 1 1 603AE044
 P 6750 5250
@@
 $EndComp
 $Comp
-L SC-STM32L412K8-rescue:Conn-My_Library-SC-STM32L412K8-rescue J6
+L SC-STM32L412K8-rescue:Conn-My_Library-SC-STM32L412K8-rescue-SC-STM32L412K8-rescue J6
 U 1 1 603AE9C5
 P 6750 5350
@@
 $EndComp
 $Comp
-L SC-STM32L412K8-rescue:Conn-My_Library-SC-STM32L412K8-rescue J3
+L SC-STM32L412K8-rescue:Conn-My_Library-SC-STM32L412K8-rescue-SC-STM32L412K8-rescue J3
 U 1 1 603B523F
 P 6750 4850
@@
 $EndComp
 $Comp
-L SC-STM32L412K8-rescue:Conn-My_Library-SC-STM32L412K8-rescue J4
+L SC-STM32L412K8-rescue:Conn-My_Library-SC-STM32L412K8-rescue-SC-STM32L412K8-rescue J4
 U 1 1 603B58EC
 P 6750 4950
@@
 Connection ~ 3850 1450
 $Comp
-L SC-STM32L412K8-rescue:Conn-My_Library-SC-STM32L412K8-rescue J2
+L SC-STM32L412K8-rescue:Conn-My_Library-SC-STM32L412K8-rescue-SC-STM32L412K8-rescue J2
 U 1 1 604E175B
 P 6150 1450
@@
 Connection ~ 7950 3750
 $Comp
-L SC-STM32L412K8-rescue:Conn-My_Library-SC-STM32L412K8-rescue J7
+L SC-STM32L412K8-rescue:Conn-My_Library-SC-STM32L412K8-rescue-SC-STM32L412K8-rescue J7
 U 1 1 60622710
 P 5200 3700
@@
 Connection ~ 5200 3600
 $Comp
-L SC-STM32L412K8-rescue:Conn-My_Library-SC-STM32L412K8-rescue J9
+L SC-STM32L412K8-rescue:Conn-My_Library-SC-STM32L412K8-rescue-SC-STM32L412K8-rescue J9
 U 1 1 6072E770
 P 6750 5450
@@
 	7500 3400 7950 3400
 $Comp
-L SC-STM32L412K8-rescue:Conn-My_Library-SC-STM32L412K8-rescue J10
+L SC-STM32L412K8-rescue:Conn-My_Library-SC-STM32L412K8-rescue-SC-STM32L412K8-rescue J10
 U 1 1 604B8416
 P 6750 5150
@@
 $EndComp
 $Comp
-L SC-STM32L412K8-rescue:Conn-My_Library-SC-STM32L412K8-rescue J11
+L SC-STM32L412K8-rescue:Conn-My_Library-SC-STM32L412K8-rescue-SC-STM32L412K8-rescue J11
 U 1 1 605058F1
 P 7250 1200
@@
 	6150 5300 6150 5500
 $Comp
-L SC-STM32L412K8-rescue:LMV7239M5-My_Library-SC-STM32L412K8-rescue U4
+L SC-STM32L412K8-rescue:LMV7239M5-My_Library-SC-STM32L412K8-rescue-SC-STM32L412K8-rescue U4
 U 1 1 6056F677
 P 6200 5050
@@
 $EndComp
 $Comp
-L SC-STM32L412K8-rescue:Conn-My_Library-SC-STM32L412K8-rescue J8
+L SC-STM32L412K8-rescue:Conn-My_Library-SC-STM32L412K8-rescue-SC-STM32L412K8-rescue J8
 U 1 1 606AB650
 P 5200 5050
@@
 $EndComp
 $Comp
-L SC-STM32L412K8-rescue:Conn-My_Library-SC-STM32L412K8-rescue J12
+L SC-STM32L412K8-rescue:Conn-My_Library-SC-STM32L412K8-rescue-SC-STM32L412K8-rescue J12
 U 1 1 60613CF0
 P 7950 2700
@@
 Buzer
 $Comp
-L SC-STM32L412K8-rescue:Conn-My_Library-SC-STM32L412K8-rescue J13
+L SC-STM32L412K8-rescue:Conn-My_Library-SC-STM32L412K8-rescue-SC-STM32L412K8-rescue J13
 U 1 1 6052B033
 P 6450 3250

Commit message: изменено:      SC-STM32L412K8/SC-STM32L412K8.sch 	изменено:      SC-STM32L412K8/SC-STM32L412K8.sch-bak 	SC-STM32L412K8/SC-STM32L412K8-rescue.dcm 	SC-STM32L412K8/SC-STM32L412K8-rescue.lib 	SC-STM32L412K8/sym-lib-table
Parts:
- L2: value 22uH -> 10uH
- R3: value 13k -> 130k
- R5: value 300k -> 3M
- U2: value LM2733YMF -> AP3015KTR
Changed lines of the file:
@@
 P 4850 2300
 F 0 "R3" H 4650 2350 50  0000 L CNN
-F 1 "13k" H 4650 2250 50  0000 L CNN
+F 1 "130k" H 4650 2250 50  0000 L CNN
 F 2 "Resistor_SMD:R_0603_1608Metric" V 4780 2300 50  0001 C CNN
 F 3 "~" H 4850 2300 50  0001 C CNN
@@
 P 4550 1450
 F 0 "L2" V 4740 1450 50  0000 C CNN
-F 1 "22uH" V 4649 1450 50  0000 C CNN
+F 1 "10uH" V 4649 1450 50  0000 C CNN
 F 2 "Inductor_SMD:L_1210_3225Metric" H 4550 1450 50  0001 C CNN
 F 3 "~" H 4550 1450 50  0001 C CNN
@@
 P 4550 1850
 F 0 "U2" H 4550 2217 50  0000 C CNN
-F 1 "LM2733YMF" H 4550 2126 50  0000 C CNN
+F 1 "AP3015KTR" H 4550 2126 50  0000 C CNN
 F 2 "Package_TO_SOT_SMD:SOT-23-5" H 4600 1600 50  0001 L CIN
 F 3 "http://www.ti.com/lit/ds/symlink/lm2733.pdf" H 4550 1950 50  0001 C CNN
@@
 P 5000 1950
 F 0 "R5" V 4793 1950 50  0000 C CNN
-F 1 "300k" V 4884 1950 50  0000 C CNN
+F 1 "3M" V 4884 1950 50  0000 C CNN
 F 2 "Resistor_SMD:R_0603_1608Metric" V 4930 1950 50  0001 C CNN
 F 3 "~" H 5000 1950 50  0001 C CNN
