File: SC-STM32L412K8/SC-STM32L412K8.sch (KiCad schematic (older format))
At the start: 72 parts, among them J1 usb, J10 PWM, J11 Vibro, J12 +3v, J13 +vibro, J2 +29.6 SiPM, J3 TxD, J4 RxD, J5 SWDIO, J6 SWCLK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

Commit message: изменено:      SC-STM32L412K8/SC-STM32L412K8.kicad_pcb 	изменено:      SC-STM32L412K8/SC-STM32L412K8.kicad_pcb-bak 	изменено:      SC-STM32L412K8/SC-STM32L412K8.net 	изменено:      SC-STM32L412K8/SC-STM32L412K8.sch 	изменено:      SC-STM32L412K8/SC-STM32L412K8.sch-bak
Parts:
- C5: value 82pF -> 1.5pF
- L2: value 10uH -> 22uH
- R19: value X -> 39k
- R20: value X -> 100k
- R3: value 130k -> 430k
- R5: value 3M -> 10M
- U3: value LTC4054ES5 -> MCP73831
Connections:
- net GND: no longer R18.1, R20.1
- net com: now reaches D6.18 (PA8)
- net com: now also R18.1, R20.1
Changed lines of the file:
@@
 P 4850 2300
 F 0 "R3" H 4650 2350 50  0000 L CNN
-F 1 "130k" H 4650 2250 50  0000 L CNN
+F 1 "430k" H 4600 2250 50  0000 L CNN
 F 2 "Resistor_SMD:R_0603_1608Metric" V 4780 2300 50  0001 C CNN
 F 3 "~" H 4850 2300 50  0001 C CNN
@@
 P 5000 2150
 F 0 "C5" V 5150 2100 50  0000 C CNN
-F 1 "82pF" V 5250 2150 50  0000 C CNN
+F 1 "1.5pF" V 5250 2150 50  0000 C CNN
 F 2 "Capacitor_SMD:C_0603_1608Metric" H 5038 2000 50  0001 C CNN
 F 3 "~" H 5000 2150 50  0001 C CNN
@@
 P 4550 1450
 F 0 "L2" V 4740 1450 50  0000 C CNN
-F 1 "10uH" V 4649 1450 50  0000 C CNN
+F 1 "22uH" V 4649 1450 50  0000 C CNN
 F 2 "Inductor_SMD:L_1210_3225Metric" H 4550 1450 50  0001 C CNN
 F 3 "~" H 4550 1450 50  0001 C CNN
@@
 P 4850 3600
 F 0 "U3" H 5200 3300 50  0000 L CNN
-F 1 "LTC4054ES5" H 4900 3200 50  0000 L CNN
+F 1 "MCP73831" H 4900 3200 50  0000 L CNN
 F 2 "Package_TO_SOT_SMD:TSOT-23-5" H 4850 3100 50  0001 C CNN
 F 3 "http://cds.linear.com/docs/en/datasheet/405442xf.pdf" H 4850 3500 50  0001 C CNN
@@
 P 5000 1950
 F 0 "R5" V 4793 1950 50  0000 C CNN
-F 1 "3M" V 4884 1950 50  0000 C CNN
+F 1 "10M" V 4884 1950 50  0000 C CNN
 F 2 "Resistor_SMD:R_0603_1608Metric" V 4930 1950 50  0001 C CNN
 F 3 "~" H 5000 1950 50  0001 C CNN
@@
 	-1   0    0    1
 $EndComp
-$Comp
-L power:GND #PWR05
-U 1 1 6057F52E
-P 8100 3400
-F 0 "#PWR05" H 8100 3150 50  0001 C CNN
-F 1 "GND" H 8105 3227 50  0001 C CNN
-F 2 "" H 8100 3400 50  0001 C CNN
-F 3 "" H 8100 3400 50  0001 C CNN
-	1    8100 3400
-	1    0    0    -1
-$EndComp
 Text GLabel 8300 3100 2    50   Input ~ 0
 tm
@@
 P 8100 1950
 F 0 "R19" H 7950 1950 50  0000 C CNN
-F 1 "X" H 7950 1850 50  0000 C CNN
+F 1 "39k" H 7950 1850 50  0000 C CNN
 F 2 "Resistor_SMD:R_0603_1608Metric" V 8030 1950 50  0001 C CNN
 F 3 "~" H 8100 1950 50  0001 C CNN
@@
 P 8100 2250
 F 0 "R20" H 7950 2350 50  0000 C CNN
-F 1 "X" H 7950 2250 50  0000 C CNN
+F 1 "100k" H 7950 2250 50  0000 C CNN
 F 2 "Resistor_SMD:R_0603_1608Metric" V 8030 2250 50  0001 C CNN
 F 3 "~" H 8100 2250 50  0001 C CNN
 	1    8100 2250
 	-1   0    0    1
-$EndComp
-$Comp
-L power:GND #PWR0104
-U 1 1 6053B5D1
-P 8100 2400
-F 0 "#PWR0104" H 8100 2150 50  0001 C CNN
-F 1 "GND" H 8105 2227 50  0001 C CNN
-F 2 "" H 8100 2400 50  0001 C CNN
-F 3 "" H 8100 2400 50  0001 C CNN
-	1    8100 2400
-	1    0    0    -1
 $EndComp
 $Comp
@@
 Wire Wire Line
 	6950 3700 7150 3700
+Text GLabel 6850 4750 0    50   Input ~ 0
+com
+Text GLabel 8050 2450 0    50   Input ~ 0
+com
+Text GLabel 8050 3500 0    50   Input ~ 0
+com
+Wire Wire Line
+	8100 2400 8100 2450
+Wire Wire Line
+	8100 2450 8050 2450
+Wire Wire Line
+	8100 3400 8100 3500
+Wire Wire Line
+	8100 3500 8050 3500
 $EndSCHEMATC
