File: SC-STM32L412K8/SC-STM32L412K8.kicad_pcb (KiCad board)
At the start: 2 copper layers, 31.6 x 15.1 mm, 59 parts, among them J1 usb, J2 +29.6, J3 TxD, J4 RxD, J5 SWDIO, J6 SWCLK, J7 +BAT, J8 SiPM-, J9 BT Status, Q1 IRLML5203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

Commit message: modified:   SC-STM32L412K8/SC-STM32L412K8-cache.lib 	modified:   SC-STM32L412K8/SC-STM32L412K8.kicad_pcb 	modified:   SC-STM32L412K8/SC-STM32L412K8.kicad_pcb-bak 	modified:   SC-STM32L412K8/SC-STM32L412K8.net 	modified:   SC-STM32L412K8/SC-STM32L412K8.sch 	modified:   SC-STM32L412K8/SC-STM32L412K8.sch-bak
Parts:
- added J10: PWM, My-library:SMD-CONN, F.Cu at (55.6, 84.4)
- moved J5 0.49 mm to (53.7, 84.4)
- moved J6 0.49 mm to (51.7, 84.4)
- moved J9 0.49 mm to (49.8, 84.4)
- moved D7 0.28 mm to (44.4, 85.3)
- moved R14 0.27 mm to (47.3, 85.3)
- moved C8 0.07 mm to (45.9, 88.7)
Connections:
- D6 pad 22: (no net) -> Net-(D6-Pad22)
Routing:
- net Net-(D6-Pad22): track 0.00 -> 8.85 mm
- net Net-(C14-Pad2): track 5.21 -> 4.40 mm

Commit message: modified:   SC-STM32L412K8/SC-STM32L412K8.kicad_pcb 	modified:   SC-STM32L412K8/SC-STM32L412K8.kicad_pcb-bak 	modified:   SC-STM32L412K8/SC-STM32L412K8.sch 	modified:   SC-STM32L412K8/SC-STM32L412K8.sch-bak
Parts:
- moved C4 1.75 mm to (52.3, 91.7)
- moved U5 1.27 mm to (53.7, 95.0)
- moved J8 1.15 mm to (56.4, 97.0)
Routing:
- net GND: track 92.9 -> 82.8 mm
- net Net-(C16-Pad1): track 17.1 -> 18.1 mm
- net +BATT: track 47.3 -> 46.4 mm

Commit message: modified:   SC-STM32L412K8/SC-STM32L412K8-cache.lib 	modified:   SC-STM32L412K8/SC-STM32L412K8.kicad_pcb 	modified:   SC-STM32L412K8/SC-STM32L412K8.kicad_pcb-bak 	modified:   SC-STM32L412K8/SC-STM32L412K8.net 	modified:   SC-STM32L412K8/SC-STM32L412K8.sch 	modified:   SC-STM32L412K8/SC-STM32L412K8.sch-bak
Parts:
- added BZ1: Buzzer, My-library:BuzerSMD, B.Cu at (31.7, 95.2)
- added J11: Vibro, My-library:SMD-CONN, F.Cu at (41.4, 96.4)
- added J12: +3v, My-library:SMD-CONN, F.Cu at (40.3, 86.2)
- added Q2: KT235, Package_TO_SOT_SMD:SOT-23, B.Cu at (36.7, 95.2)
- added Q3: KT235, Package_TO_SOT_SMD:SOT-23, F.Cu at (39.7, 96.3)
- added R15: 4.7k, Resistor_SMD:R_0603_1608Metric, B.Cu at (39.0, 95.2)
- added R16: 4.7k, Resistor_SMD:R_0603_1608Metric, F.Cu at (38.7, 93.4)
- moved C13 3.06 mm to (34.2, 91.2), turned to 90 degrees
- moved C3 2.53 mm to (37.3, 92.0), turned to 180 degrees
- moved J5 2.17 mm to (51.5, 84.4)
- moved J6 1.69 mm to (53.4, 84.4)
- moved J7 0.49 mm to (36.0, 86.4)
- moved R12 0.37 mm to (34.4, 85.5)
- moved C10 0.25 mm to (32.7, 85.5)
- moved J10 0.25 mm to (55.3, 84.4)
- moved J9 0.25 mm to (49.6, 84.4)
- moved R7 0.17 mm to (53.5, 87.9)
- moved R6 0.06 mm to (35.3, 91.4)
Connections:
- D6 pad 10: (no net) -> Buzer
- D6 pad 7: (no net) -> Vibro
Routing:
- net GND: track 82.8 -> 155.3 mm, vias 7 -> 9
- net +BATT: track 46.4 -> 57.6 mm
- net Buzer: track 0.00 -> 6.86 mm, vias 0 -> 1
- net Vibro: track 0.00 -> 3.74 mm
- net Net-(BZ1-Pad2): track 0.00 -> 1.76 mm
- net Net-(Q2-Pad1): track 0.00 -> 1.52 mm
- net Net-(C16-Pad1): track 18.1 -> 19.6 mm
- net Net-(D6-Pad24): track 4.52 -> 5.94 mm
- net Net-(Q3-Pad1): track 0.00 -> 1.12 mm
- net Net-(C13-Pad1): track 8.89 -> 9.73 mm

Commit message: modified:   SC-STM32L412K8/SC-STM32L412K8.kicad_pcb 	modified:   SC-STM32L412K8/SC-STM32L412K8.kicad_pcb-bak 	modified:   SC-STM32L412K8/SC-STM32L412K8.net 	modified:   SC-STM32L412K8/SC-STM32L412K8.sch 	modified:   SC-STM32L412K8/SC-STM32L412K8.sch-bak 	modified:   STM32Code/.settings/language.settings.xml 	modified:   STM32Code/Core/Src/main.c 	modified:   STM32Code/Release/Core/Src/main.o 	modified:   STM32Code/Release/Core/Src/main.su 	modified:   STM32Code/Release/SC4-LCD128x32.bin 	modified:   STM32Code/Release/SC4-LCD128x32.elf 	modified:   STM32Code/Release/SC4-LCD128x32.list 	modified:   STM32Code/Release/SC4-LCD128x32.map 	modified:   STM32Code/Release/makefile
Parts:
- added J13: +vibro, My-library:SMD-CONN, F.Cu at (28.2, 84.3)
- added R17: X, Resistor_SMD:R_0603_1608Metric, B.Cu at (48.5, 95.4)
- added R18: X, Resistor_SMD:R_0603_1608Metric, B.Cu at (48.4, 94.1)
- J2: value +29.6 -> +29.6 SiPM
- moved R14 0.22 mm to (47.3, 85.6)
- moved J9 0.22 mm to (49.3, 84.4)
- moved J5 0.21 mm to (51.3, 84.4)
- moved J6 0.21 mm to (53.2, 84.4)
- moved J10 0.20 mm to (55.1, 84.4)
Connections:
- D6 pad 14: (no net) -> tm
Routing:
- net GND: track 155.3 -> 161.9 mm
- net +BATT: track 57.6 -> 61.1 mm, vias 0 -> 1
- net tm: track 0.00 -> 2.59 mm, vias 0 -> 1
- net Net-(C16-Pad1): track 19.6 -> 21.7 mm
- net Net-(D6-Pad24): track 5.94 -> 5.26 mm

Commit message: modified:   SC-STM32L412K8/SC-STM32L412K8.kicad_pcb 	modified:   SC-STM32L412K8/SC-STM32L412K8.kicad_pcb-bak 	modified:   SC-STM32L412K8/SC-STM32L412K8.net 	modified:   SC-STM32L412K8/SC-STM32L412K8.sch 	modified:   SC-STM32L412K8/SC-STM32L412K8.sch-bak
Parts:
- added R19: X, Resistor_SMD:R_0603_1608Metric, B.Cu at (56.9, 94.7)
- added R20: X, Resistor_SMD:R_0603_1608Metric, B.Cu at (47.8, 93.8)
- moved R17 3.94 mm to (52.4, 95.7), turned to 90 degrees
- moved R18 2.16 mm to (49.1, 96.1), turned to 90 degrees
- moved U5 1.56 mm to (54.8, 96.1)
- moved R15 1.35 mm to (40.2, 95.8), turned to 0 degrees
- moved C15 1.23 mm to (57.5, 96.8)
- moved BZ1 0.62 mm to (31.6, 95.8)
Connections:
- D6 pad 12: (no net) -> tm
- D6 pad 13: (no net) -> bl
- D6 pad 14: tm -> (no net)
Routing:
- net bl: track 0.00 -> 11.3 mm, vias 0 -> 1
- net tm: track 2.59 -> 9.80 mm
- net Buzer: track 6.86 -> 4.95 mm
- net GND: track 161.9 -> 162.9 mm
- net Net-(Q2-Pad1): track 1.52 -> 2.40 mm
- net +BATT: track 61.1 -> 61.9 mm

Commit message: изменено:      SC-STM32L412K8/SC-STM32L412K8-cache.lib 	изменено:      SC-STM32L412K8/SC-STM32L412K8.kicad_pcb 	изменено:      SC-STM32L412K8/SC-STM32L412K8.kicad_pcb-bak 	изменено:      SC-STM32L412K8/SC-STM32L412K8.sch 	изменено:      SC-STM32L412K8/SC-STM32L412K8.sch-bak 	SC-STM32L412K8/SC-STM32L412K8-rescue.dcm 	SC-STM32L412K8/SC-STM32L412K8-rescue.lib
Parts:
- moved C15 30.5 mm to (57.8, 66.3)
- moved C19 30.5 mm to (51.1, 65.5)
- moved C20 30.5 mm to (40.1, 60.1)
- moved C9 30.5 mm to (56.0, 57.7)
- moved D1 30.5 mm to (30.8, 65.6)
- moved J11 30.5 mm to (41.7, 65.9)
- moved J3 30.5 mm to (53.3, 65.4)
- moved L1 30.5 mm to (34.0, 55.0)
- moved Q2 30.5 mm to (37.0, 64.7)
- moved Q3 30.5 mm to (40.0, 65.7)
- moved R1 30.5 mm to (34.0, 65.4)
- moved R11 30.5 mm to (49.2, 55.2)
- moved R13 30.5 mm to (52.2, 55.2)
- moved R15 30.5 mm to (40.5, 65.3)
- moved R8 30.5 mm to (58.1, 59.0)
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
Commit message: изменено:      SC-STM32L412K8/SC-STM32L412K8.kicad_pcb 	изменено:      SC-STM32L412K8/SC-STM32L412K8.kicad_pcb-bak 	изменено:      SC-STM32L412K8/SC-STM32L412K8.net 	изменено:      SC-STM32L412K8/SC-STM32L412K8.sch 	изменено:      SC-STM32L412K8/SC-STM32L412K8.sch-bak
Parts:
- C5: value 82pF -> 1.5pF
- R19: value X -> 39k
- R20: value X -> 100k
- R3: value 13k -> 430k
- R5: value 300k -> 10M
- U2: value LM2733YMF -> AP3015KTR
- U3: value LTC4054ES5 -> MCP73831
- moved R17 3.88 mm to (48.8, 65.3), turned to 0 degrees
- moved R18 2.32 mm to (49.5, 63.2), turned to 270 degrees
- moved U5 1.37 mm to (53.8, 65.6)
- moved R19 0.95 mm to (56.3, 64.2)
Connections:
- D6 pad 18: (no net) -> com
- R18 pad 1: GND -> com
- R20 pad 1: GND -> com
Routing:
- net GND: track 162.9 -> 171.4 mm
- net com: track 0.00 -> 4.40 mm, vias 0 -> 1
- net tm: track 9.80 -> 6.81 mm
- net +BATT: track 61.9 -> 64.3 mm
- net bl: track 11.3 -> 10.8 mm
