File: SC-STM32L412K8/SC-STM32L412K8.kicad_pcb (KiCad board)
At the start: 2 copper layers, 31.6 x 15.1 mm, 72 parts, among them J1 usb, J10 PWM, J11 Vibro, J12 +3v, J13 +vibro, J2 +29.6 SiPM, J3 TxD, J4 RxD, J5 SWDIO, J6 SWCLK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

Commit message: modified:   SC-STM32L412K8/SC-STM32L412K8-cache.lib 	modified:   SC-STM32L412K8/SC-STM32L412K8.kicad_pcb 	modified:   SC-STM32L412K8/SC-STM32L412K8.kicad_pcb-bak 	modified:   SC-STM32L412K8/SC-STM32L412K8.net 	modified:   SC-STM32L412K8/SC-STM32L412K8.sch 	modified:   SC-STM32L412K8/SC-STM32L412K8.sch-bak
Parts:
- R3: value 13k -> 430k
- R5: value 300k -> 10M
- U2: value LM2733YMF -> AP3015KTR
- moved R18 4.89 mm to (45.0, 63.5), turned to 0 degrees
- moved R17 3.95 mm to (48.8, 64.8), turned to 0 degrees
- moved U5 1.44 mm to (53.7, 65.5)
- moved R20 0.97 mm to (47.3, 62.8)
Routing:
- net tm: track 9.80 -> 4.48 mm
- net +BATT: track 61.9 -> 63.3 mm
- net GND: track 162.9 -> 163.7 mm
