File: SC-STM32L412K8-light/SC-STM32L412K8.kicad_pcb (KiCad board)
At the start: 2 copper layers, 31.6 x 15.1 mm, 65 parts, among them J1 usb, J11 Vibro, J12 +3v, J13 +vibro, J2 +29.6 SiPM, J3 TxD, J4 RxD, J5 SWDIO, J6 SWCLK, J7 +BAT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

Commit message: изменено:      SC-STM32L412K8-light/SC-STM32L412K8-cache.lib 	изменено:      SC-STM32L412K8-light/SC-STM32L412K8.kicad_pcb 	изменено:      SC-STM32L412K8-light/SC-STM32L412K8.kicad_pcb-bak 	изменено:      SC-STM32L412K8-light/SC-STM32L412K8.net 	изменено:      SC-STM32L412K8-light/SC-STM32L412K8.sch 	изменено:      SC-STM32L412K8-light/SC-STM32L412K8.sch-bak
Parts:
- removed C4: 0.1uF, Capacitor_SMD:C_0603_1608Metric
- removed U1: LP2985-3.0, Package_TO_SOT_SMD:SOT-23-5
- moved C15 8.98 mm to (56.9, 57.4), turned to 180 degrees
- moved U5 6.56 mm to (56.9, 59.8)
- moved C2 4.21 mm to (53.4, 60.4), turned to 270 degrees
- moved R17 3.55 mm to (47.1, 61.6), turned to 90 degrees
- moved R19 2.77 mm to (54.0, 65.8)
- moved R18 0.96 mm to (48.6, 62.5), turned to 270 degrees
- moved C8 0.94 mm to (46.2, 57.4)
- moved C6 0.83 mm to (48.1, 57.4)
- moved C11 0.72 mm to (49.9, 57.4)
- moved C14 0.62 mm to (51.7, 57.4)
- moved J2 0.53 mm to (53.8, 55.2)
- moved R20 0.43 mm to (50.0, 62.5)
- moved C19 0.21 mm to (51.0, 65.7)
Connections:
- C16 pad 1: Net-(C16-Pad1) -> Net-(C12-Pad1)
- C17 pad 1: Net-(C16-Pad1) -> Net-(C12-Pad1)
- C19 pad 1: Net-(C16-Pad1) -> Net-(C12-Pad1)
- C2 pad 1: +BATT -> Net-(C12-Pad1)
- D6 pad 1: Net-(C16-Pad1) -> Net-(C12-Pad1)
- D6 pad 17: Net-(C16-Pad1) -> Net-(C12-Pad1)
- J12 pad 1: Net-(C16-Pad1) -> Net-(C12-Pad1)
- L4 pad 1: Net-(C16-Pad1) -> Net-(C12-Pad1)
- R17 pad 2: Net-(C16-Pad1) -> Net-(C12-Pad1)
- U5 pad 2: Net-(C16-Pad1) -> Net-(C12-Pad1)
Routing:
- net Net-(C12-Pad1): track 2.92 -> 35.7 mm, vias 1 -> 3
- net Net-(C16-Pad1): track 21.4 -> 0.00 mm, vias 1 -> 0
- net GND: track 178.1 -> 164.7 mm, vias 8 -> 9
- net +BATT: track 64.3 -> 60.4 mm
- net Net-(C4-Pad1): track 1.37 -> 0.00 mm
- net Net-(C14-Pad2): track 4.23 -> 3.18 mm
- net bl: track 10.1 -> 10.7 mm

Commit message: modified:   SC-STM32L412K8-light/SC-STM32L412K8.kicad_pcb 	modified:   SC-STM32L412K8-light/SC-STM32L412K8.kicad_pcb-bak 	modified:   SC-STM32L412K8-light/SC-STM32L412K8.net 	modified:   SC-STM32L412K8-light/SC-STM32L412K8.sch 	modified:   SC-STM32L412K8-light/SC-STM32L412K8.sch-bak 	modified:   STM32L412K8code/.settings/language.settings.xml
Parts:
- removed R17, R18: X, Resistor_SMD:R_0603_1608Metric
- added C4: 22uF, Capacitor_SMD:C_0805_2012Metric, F.Cu at (33.2, 55.2)
- L1: value 10uH -> LQM21FN100N
- L2: value 22uH -> LQH31MN220J03L
- L3, L4: value 47uH -> MLZ2012M470WT000
- Q2, Q3: value KT235 -> KT231Г9
- moved R19 5.47 mm to (48.7, 64.5), turned to 270 degrees
- moved R20 3.60 mm to (46.6, 63.7), turned to 0 degrees
- moved R4 2.08 mm to (35.6, 55.2)
- moved J7 0.42 mm to (36.0, 56.9)
- moved R6 0.27 mm to (33.5, 57.5)
- moved C15 0.16 mm to (57.1, 57.3)
Connections:
- D6 pad 12: tm -> com
- D6 pad 18: com -> (no net)
Routing:
- net GND: track 164.7 -> 174.4 mm, vias 9 -> 10
- net bl: track 10.7 -> 2.99 mm
- net tm: track 5.98 -> 0.00 mm, vias 1 -> 0
- net +BATT: track 60.4 -> 65.6 mm
- net Net-(D1-Pad2): track 3.82 -> 1.58 mm
- net com: track 3.18 -> 1.59 mm
- net Net-(C4-Pad2): track 3.46 -> 4.62 mm
- net Net-(C13-Pad1): track 14.0 -> 13.2 mm
- net Net-(C12-Pad1): track 35.7 -> 35.2 mm, vias 3 -> 2
