File: SC-STM32L412K8-light/SC-STM32L412K8.sch (KiCad schematic (older format))
At the start: 65 parts, among them J1 usb, J11 Vibro, J12 +3v, J13 +vibro, J2 +29.6 SiPM, J3 TxD, J4 RxD, J5 SWDIO, J6 SWCLK, J7 +BAT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

Commit message: изменено:      SC-STM32L412K8-light/SC-STM32L412K8-cache.lib 	изменено:      SC-STM32L412K8-light/SC-STM32L412K8.kicad_pcb 	изменено:      SC-STM32L412K8-light/SC-STM32L412K8.kicad_pcb-bak 	изменено:      SC-STM32L412K8-light/SC-STM32L412K8.net 	изменено:      SC-STM32L412K8-light/SC-STM32L412K8.sch 	изменено:      SC-STM32L412K8-light/SC-STM32L412K8.sch-bak
Parts:
- removed C4: 0.1uF, Capacitor_SMD:C_0603_1608Metric, symbol Device:C
- removed U1: LP2985-3.0, Package_TO_SOT_SMD:SOT-23-5, symbol Regulator_Linear:LP2985-3.0
Connections:
- wire segments 108 -> 103
Other:
- moved on the sheet: C13, C15, C19, C2, C5, D1, J1, R1, R15, R16, R17, R18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

Commit message: modified:   SC-STM32L412K8-light/SC-STM32L412K8.kicad_pcb 	modified:   SC-STM32L412K8-light/SC-STM32L412K8.kicad_pcb-bak 	modified:   SC-STM32L412K8-light/SC-STM32L412K8.net 	modified:   SC-STM32L412K8-light/SC-STM32L412K8.sch 	modified:   SC-STM32L412K8-light/SC-STM32L412K8.sch-bak 	modified:   STM32L412K8code/.settings/language.settings.xml
Parts:
- removed R17, R18: X, Resistor_SMD:R_0603_1608Metric, symbol Device:R
- added C4: 22uF, Capacitor_SMD:C_0805_2012Metric, symbol Device:C
- L1: value 10uH -> LQM21FN100N
- L2: value 22uH -> LQH31MN220J03L
- L3, L4: value 47uH -> MLZ2012M470WT000
- Q2, Q3: value KT235 -> KT231Г9
Connections:
- net labels removed: tm
- wire segments 103 -> 102
Other:
- note added: "C1, C2, C3, C4, C12, C13, C15, C16, C17, C18, C19 GRM21BR60J226M"
- moved on the sheet: C12, C15, C19, J1, R15, R16, R19, R20, R6, U5

Commit message: изменено:      SC-STM32L412K8-light/SC-STM32L412K8.kicad_pcb 	изменено:      SC-STM32L412K8-light/SC-STM32L412K8.kicad_pcb-bak 	изменено:      SC-STM32L412K8-light/SC-STM32L412K8.net 	изменено:      SC-STM32L412K8-light/SC-STM32L412K8.sch 	изменено:      SC-STM32L412K8-light/SC-STM32L412K8.sch-bak 	изменено:      STM32L412K8code/Release/Core/Src/stm32l4xx_it.su
Parts:
- added R10: 3k*, Resistor_SMD:R_0603_1608Metric, symbol Device:R
Connections:
- wire segments 102 -> 104
Other:
- moved on the sheet: C1, C11, C14, C3, C5, C6, C7, C8, D2, L1, L2, L3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

Commit message: изменено:      SC-STM32L412K8-light/SC-STM32L412K8-cache.lib 	изменено:      SC-STM32L412K8-light/SC-STM32L412K8.kicad_pcb 	изменено:      SC-STM32L412K8-light/SC-STM32L412K8.kicad_pcb-bak 	изменено:      SC-STM32L412K8-light/SC-STM32L412K8.net 	изменено:      SC-STM32L412K8-light/SC-STM32L412K8.sch 	изменено:      SC-STM32L412K8-light/SC-STM32L412K8.sch-bak
Parts:
- removed BZ1: Buzzer, My-library:BuzerSMD, symbol Device:Buzzer
- removed Q2, Q3: KT231Г9, Package_TO_SOT_SMD:SOT-23, symbol Device:Q_NPN_BEC
- added J10: Buzzer, My-library:SMD-CONN, symbol SC-STM32L412K8-rescue:Conn-My_Library-SC-STM32L412K8-rescue-SC-STM32L412K8-resc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
- added Q1, Q2: 2N7002, Package_TO_SOT_SMD:SOT-23, symbol Transistor_FET:2N7002
- added R12: 200, Resistor_SMD:R_0603_1608Metric, symbol Device:R
- R15, R16: value 4.7k -> 100k
Connections:
- wire segments 104 -> 110
Other:
- moved on the sheet: R15, R16
Changed lines of the file:
@@
 Connection ~ 7050 2800
-$Comp
-L Device:Q_NPN_BEC Q2
-U 1 1 604F8B65
-P 7550 2400
-F 0 "Q2" H 7741 2446 50  0000 L CNN
-F 1 "KT231Г9" H 7741 2355 50  0000 L CNN
-F 2 "Package_TO_SOT_SMD:SOT-23" H 7750 2500 50  0001 C CNN
-F 3 "~" H 7550 2400 50  0001 C CNN
-	1    7550 2400
-	1    0    0    -1
-$EndComp
-$Comp
-L Device:Q_NPN_BEC Q3
-U 1 1 604F994F
-P 7550 1600
-F 0 "Q3" H 7750 1650 50  0000 L CNN
-F 1 "KT231Г9" H 7750 1550 50  0000 L CNN
-F 2 "Package_TO_SOT_SMD:SOT-23" H 7750 1700 50  0001 C CNN
-F 3 "~" H 7550 1600 50  0001 C CNN
-	1    7550 1600
-	1    0    0    -1
-$EndComp
 $Comp
 L Device:R R15
 U 1 1 604FA546
-P 7200 2400
-F 0 "R15" V 7000 2400 50  0000 C CNN
-F 1 "4.7k" V 7100 2400 50  0000 C CNN
-F 2 "Resistor_SMD:R_0603_1608Metric" V 7130 2400 50  0001 C CNN
-F 3 "~" H 7200 2400 50  0001 C CNN
-	1    7200 2400
-	0    1    1    0
+P 7500 2400
+F 0 "R15" H 7800 2400 50  0000 C CNN
+F 1 "100k" H 7750 2500 50  0000 C CNN
+F 2 "Resistor_SMD:R_0603_1608Metric" V 7430 2400 50  0001 C CNN
+F 3 "~" H 7500 2400 50  0001 C CNN
+	1    7500 2400
+	-1   0    0    1
 $EndComp
 $Comp
 L Device:R R16
 U 1 1 604FB12B
-P 7200 1600
-F 0 "R16" V 7000 1600 50  0000 C CNN
-F 1 "4.7k" V 7100 1600 50  0000 C CNN
-F 2 "Resistor_SMD:R_0603_1608Metric" V 7130 1600 50  0001 C CNN
-F 3 "~" H 7200 1600 50  0001 C CNN
-	1    7200 1600
-	0    1    1    0
+P 7500 1550
+F 0 "R16" H 7700 1550 50  0000 C CNN
+F 1 "100k" H 7700 1650 50  0000 C CNN
+F 2 "Resistor_SMD:R_0603_1608Metric" V 7430 1550 50  0001 C CNN
+F 3 "~" H 7500 1550 50  0001 C CNN
+	1    7500 1550
+	-1   0    0    1
 $EndComp
 $Comp
 L power:GND #PWR0101
 U 1 1 604FBD4D
-P 7650 2600
-F 0 "#PWR0101" H 7650 2350 50  0001 C CNN
-F 1 "GND" H 7655 2427 50  0001 C CNN
-F 2 "" H 7650 2600 50  0001 C CNN
-F 3 "" H 7650 2600 50  0001 C CNN
-	1    7650 2600
+P 7800 2550
+F 0 "#PWR0101" H 7800 2300 50  0001 C CNN
+F 1 "GND" H 7805 2377 50  0001 C CNN
+F 2 "" H 7800 2550 50  0001 C CNN
+F 3 "" H 7800 2550 50  0001 C CNN
+	1    7800 2550
 	1    0    0    -1
 $EndComp
@@
 L power:GND #PWR0102
 U 1 1 604FC90E
-P 7650 1800
-F 0 "#PWR0102" H 7650 1550 50  0001 C CNN
-F 1 "GND" H 7655 1627 50  0001 C CNN
-F 2 "" H 7650 1800 50  0001 C CNN
-F 3 "" H 7650 1800 50  0001 C CNN
-	1    7650 1800
-	1    0    0    -1
-$EndComp
-$Comp
-L Device:Buzzer BZ1
-U 1 1 604FDD84
-P 7750 2100
-F 0 "BZ1" H 7902 2129 50  0000 L CNN
-F 1 "Buzzer" H 7902 2038 50  0000 L CNN
-F 2 "My-library:BuzerSMD" V 7725 2200 50  0001 C CNN
-F 3 "~" V 7725 2200 50  0001 C CNN
-	1    7750 2100
-	1    0    0    -1
-$EndComp
-$Comp
-L power:+BATT #PWR0103
-U 1 1 60504BD6
-P 7650 2000
-F 0 "#PWR0103" H 7650 1850 50  0001 C CNN
-F 1 "+BATT" V 7650 2250 50  0000 C CNN
-F 2 "" H 7650 2000 50  0001 C CNN
-F 3 "" H 7650 2000 50  0001 C CNN
-	1    7650 2000
-	0    -1   -1   0
+P 7800 1700
+F 0 "#PWR0102" H 7800 1450 50  0001 C CNN
+F 1 "GND" H 7805 1527 50  0001 C CNN
+F 2 "" H 7800 1700 50  0001 C CNN
+F 3 "" H 7800 1700 50  0001 C CNN
+	1    7800 1700
+	1    0    0    -1
 $EndComp
 $Comp
 L SC-STM32L412K8-rescue:Conn-My_Library-SC-STM32L412K8-rescue-SC-STM32L412K8-rescue-SC-STM32L412K8-rescue J11
 U 1 1 605058F1
-P 7750 1400
-F 0 "J11" H 7692 1175 50  0001 C CNN
-F 1 "Vibro" H 7750 1500 50  0000 C CNN
-F 2 "My-library:SMD-CONN" H 7750 1400 50  0001 C CNN
-F 3 "~" H 7750 1400 50  0001 C CNN
-	1    7750 1400
+P 7900 1200
+F 0 "J11" H 7842 975 50  0001 C CNN
+F 1 "Vibro" H 7900 1300 50  0000 C CNN
+F 2 "My-library:SMD-CONN" H 7900 1200 50  0001 C CNN
+F 3 "~" H 7900 1200 50  0001 C CNN
+	1    7900 1200
 	1    0    0    -1
 $EndComp
@@
 	0    -1   -1   0
 $EndComp
-Text GLabel 7050 1600 0    50   Input ~ 0
+Text GLabel 7350 1400 0    50   Input ~ 0
 Vibro
 Text GLabel 6850 4050 0    50   Input ~ 0
 Vibro
-Text GLabel 7050 2400 0    50   Input ~ 0
+Text GLabel 7350 2250 0    50   Input ~ 0
 Buzer
 Text GLabel 6850 4250 0    50   Input ~ 0
@@
 Wire Wire Line
 	5500 5150 5500 5100
-Text Notes 5250 1150 0    50   ~ 0
+Text Notes 5400 950  0    50   ~ 0
 C6, C7, C8, C11, C14 GRM21BC8YA106KE11L
 Wire Wire Line
@@
 Wire Wire Line
 	3900 1400 3900 2200
+$Comp
+L Device:R R12
+U 1 1 60985878
+P 7950 2050
+F 0 "R12" V 7750 2050 50  0000 C CNN
+F 1 "200" V 7850 2050 50  0000 C CNN
+F 2 "Resistor_SMD:R_0603_1608Metric" V 7880 2050 50  0001 C CNN
+F 3 "~" H 7950 2050 50  0001 C CNN
+	1    7950 2050
+	0    1    1    0
+$EndComp
+$Comp
+L SC-STM32L412K8-rescue:Conn-My_Library-SC-STM32L412K8-rescue-SC-STM32L412K8-rescue-SC-STM32L412K8-rescue J10
+U 1 1 6098637F
+P 8200 2050
+F 0 "J10" H 8142 1825 50  0001 C CNN
+F 1 "Buzzer" H 8200 2150 50  0000 C CNN
+F 2 "My-library:SMD-CONN" H 8200 2050 50  0001 C CNN
+F 3 "~" H 8200 2050 50  0001 C CNN
+	1    8200 2050
+	1    0    0    -1
+$EndComp
+$Comp
+L Transistor_FET:2N7002 Q1
+U 1 1 609A9FBA
+P 7700 1400
+F 0 "Q1" H 7906 1446 50  0000 L CNN
+F 1 "2N7002" H 7906 1355 50  0000 L CNN
+F 2 "Package_TO_SOT_SMD:SOT-23" H 7900 1325 50  0001 L CIN
+F 3 "https://www.fairchildsemi.com/datasheets/2N/2N7002.pdf" H 7700 1400 50  0001 L CNN
+	1    7700 1400
+	1    0    0    -1
+$EndComp
+Wire Wire Line
+	7800 1600 7800 1700
+Wire Wire Line
+	7500 1700 7800 1700
+Connection ~ 7800 1700
+Wire Wire Line
+	7350 1400 7500 1400
+Connection ~ 7500 1400
+$Comp
+L Transistor_FET:2N7002 Q2
+U 1 1 609E193B
+P 7700 2250
+F 0 "Q2" H 7906 2296 50  0000 L CNN
+F 1 "2N7002" H 7906 2205 50  0000 L CNN
+F 2 "Package_TO_SOT_SMD:SOT-23" H 7900 2175 50  0001 L CIN
+F 3 "https://www.fairchildsemi.com/datasheets/2N/2N7002.pdf" H 7700 2250 50  0001 L CNN
+	1    7700 2250
+	1    0    0    -1
+$EndComp
+Wire Wire Line
+	7350 2250 7500 2250
+Connection ~ 7500 2250
+Wire Wire Line
+	7500 2550 7800 2550
+Wire Wire Line
+	7800 2550 7800 2450
+Connection ~ 7800 2550
 $EndSCHEMATC

Commit message: изменено:      SC-STM32L412K8-light/SC-STM32L412K8.sch 	изменено:      SC-STM32L412K8-light/SC-STM32L412K8.sch-bak 	изменено:      STM32L412K8code/Release/Core/Src/main.su
Parts:
- J3: value TxD -> TxD (20)
- J4: value RxD -> RxD (19)
Changed lines of the file:
@@
 P 6750 4850
 F 0 "J3" H 6692 4625 50  0001 C CNN
-F 1 "TxD" H 6850 4850 50  0000 C CNN
+F 1 "TxD (20)" H 6900 4850 50  0000 C CNN
 F 2 "My-library:SMD-CONN" H 6750 4850 50  0001 C CNN
 F 3 "~" H 6750 4850 50  0001 C CNN
@@
 P 6750 4950
 F 0 "J4" H 6692 4725 50  0001 C CNN
-F 1 "RxD" H 6850 4950 50  0000 C CNN
+F 1 "RxD (19)" H 6900 4950 50  0000 C CNN
 F 2 "My-library:SMD-CONN" H 6750 4950 50  0001 C CNN
 F 3 "~" H 6750 4950 50  0001 C CNN

Commit message: modified:   FreeCAD/sc-box-7.FCStd 	modified:   FreeCAD/sc-box-7.stl 	modified:   FreeCAD/sc-cover-7.FCStd 	modified:   FreeCAD/sc-cover-7.FCStd1 	modified:   FreeCAD/sc-cover-7.stl 	modified:   SC-STM32L412K8-light/SC-STM32L412K8.kicad_pcb 	modified:   SC-STM32L412K8-light/SC-STM32L412K8.kicad_pcb-bak 	modified:   SC-STM32L412K8-light/SC-STM32L412K8.net 	modified:   SC-STM32L412K8-light/SC-STM32L412K8.sch 	modified:   SC-STM32L412K8-light/SC-STM32L412K8.sch-bak
Parts:
- Q1, Q2: value 2N7002 -> IRLML6344
- R8: value 4.7k -> 5.1k
Other:
- moved on the sheet: C11, C14, C5, C6, C7, C8, D2, L1, L2, L3, R11, R13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

Commit message: изменено:      AndroidDoZer/app/src/main/java/ru/starline/dozer/FullscreenActivity2.java 	изменено:      AndroidDoZer/app/src/main/res/layout/activity_fullscreen2.xml 	изменено:      SC-STM32L412K8-light/SC-STM32L412K8-cache.lib 	изменено:      SC-STM32L412K8-light/SC-STM32L412K8.kicad_pcb 	изменено:      SC-STM32L412K8-light/SC-STM32L412K8.kicad_pcb-bak 	изменено:      SC-STM32L412K8-light/SC-STM32L412K8.net 	изменено:      SC-STM32L412K8-light/SC-STM32L412K8.sch 	изменено:      SC-STM32L412K8-light/SC-STM32L412K8.sch-bak 	изменено:      STM32L412K8code/.settings/language.settings.xml
Parts:
- added D3: LTC1662CMS8, Package_SO:MSOP-8_3x3mm_P0.65mm, symbol My_Library:LTC1661CMS8
- added R17: X, Resistor_SMD:R_0603_1608Metric, symbol Device:R
Connections:
- net GND: now also D3.7 (Gnd)
- net +3V3: now reaches C12.1, C16.1, C17.1, C19.1, C2.1, D6.1 (Vdd), D6.17 (Vdd), J12.1 (Pin_1), L4.1, R7.1, U4.5 (V+), U5.2 (VO)
- net +3V3: now also D3.4 (REF), D3.6 (Vcc)
- net DI: now reaches D6.18 (PA8)
- net DI: now also D3.3 (SDI)
- net CS: now reaches D6.22 (PA12)
- net CS: now also D3.1 (CS/LD)
- net SC: now reaches D6.27 (PB4)
- net SC: now also D3.2 (SCK)
- net Adjust: now reaches R10.1, R3.2
- net Adjust: now also R17.2
- new net: D3.5 (VoutB), R17.1
Other:
- moved on the sheet: Q1, Q2, R12, R15, R16
Changed lines of the file:
@@
 L Device:R R15
 U 1 1 604FA546
-P 7500 2400
-F 0 "R15" H 7650 2350 50  0000 C CNN
-F 1 "100k" H 7650 2450 50  0000 C CNN
-F 2 "Resistor_SMD:R_0603_1608Metric" V 7430 2400 50  0001 C CNN
-F 3 "~" H 7500 2400 50  0001 C CNN
-	1    7500 2400
+P 4350 5350
+F 0 "R15" H 4500 5300 50  0000 C CNN
+F 1 "100k" H 4500 5400 50  0000 C CNN
+F 2 "Resistor_SMD:R_0603_1608Metric" V 4280 5350 50  0001 C CNN
+F 3 "~" H 4350 5350 50  0001 C CNN
+	1    4350 5350
 	-1   0    0    1
 $EndComp
@@
 L Device:R R16
 U 1 1 604FB12B
-P 7500 1550
-F 0 "R16" H 7650 1500 50  0000 C CNN
-F 1 "100k" H 7650 1600 50  0000 C CNN
-F 2 "Resistor_SMD:R_0603_1608Metric" V 7430 1550 50  0001 C CNN
-F 3 "~" H 7500 1550 50  0001 C CNN
-	1    7500 1550
+P 4350 4500
+F 0 "R16" H 4500 4450 50  0000 C CNN
+F 1 "100k" H 4500 4550 50  0000 C CNN
+F 2 "Resistor_SMD:R_0603_1608Metric" V 4280 4500 50  0001 C CNN
+F 3 "~" H 4350 4500 50  0001 C CNN
+	1    4350 4500
 	-1   0    0    1
 $EndComp
@@
 L power:GND #PWR0101
 U 1 1 604FBD4D
-P 7800 2550
-F 0 "#PWR0101" H 7800 2300 50  0001 C CNN
-F 1 "GND" H 7805 2377 50  0001 C CNN
-F 2 "" H 7800 2550 50  0001 C CNN
-F 3 "" H 7800 2550 50  0001 C CNN
-	1    7800 2550
+P 4650 5500
+F 0 "#PWR0101" H 4650 5250 50  0001 C CNN
+F 1 "GND" H 4655 5327 50  0001 C CNN
+F 2 "" H 4650 5500 50  0001 C CNN
+F 3 "" H 4650 5500 50  0001 C CNN
+	1    4650 5500
 	1    0    0    -1
 $EndComp
@@
 L power:GND #PWR0102
 U 1 1 604FC90E
-P 7800 1700
-F 0 "#PWR0102" H 7800 1450 50  0001 C CNN
-F 1 "GND" H 7805 1527 50  0001 C CNN
-F 2 "" H 7800 1700 50  0001 C CNN
-F 3 "" H 7800 1700 50  0001 C CNN
-	1    7800 1700
+P 4650 4650
+F 0 "#PWR0102" H 4650 4400 50  0001 C CNN
+F 1 "GND" H 4655 4477 50  0001 C CNN
+F 2 "" H 4650 4650 50  0001 C CNN
+F 3 "" H 4650 4650 50  0001 C CNN
+	1    4650 4650
 	1    0    0    -1
 $EndComp
@@
 L SC-STM32L412K8-rescue:Conn-My_Library-SC-STM32L412K8-rescue-SC-STM32L412K8-rescue-SC-STM32L412K8-rescue J11
 U 1 1 605058F1
-P 7900 1200
-F 0 "J11" H 7842 975 50  0001 C CNN
-F 1 "Vibro" H 7900 1300 50  0000 C CNN
-F 2 "My-library:SMD-CONN" H 7900 1200 50  0001 C CNN
-F 3 "~" H 7900 1200 50  0001 C CNN
-	1    7900 1200
+P 4750 4150
+F 0 "J11" H 4692 3925 50  0001 C CNN
+F 1 "Vibro" H 4750 4250 50  0000 C CNN
+F 2 "My-library:SMD-CONN" H 4750 4150 50  0001 C CNN
+F 3 "~" H 4750 4150 50  0001 C CNN
+	1    4750 4150
 	1    0    0    -1
 $EndComp
@@
 	0    -1   -1   0
 $EndComp
-Text GLabel 7350 1400 0    50   Input ~ 0
+Text GLabel 4200 4350 0    50   Input ~ 0
 Vibro
 Text GLabel 6850 4050 0    50   Input ~ 0
 Vibro
-Text GLabel 7350 2250 0    50   Input ~ 0
+Text GLabel 4200 5200 0    50   Input ~ 0
 Buzer
 Text GLabel 6850 4250 0    50   Input ~ 0
@@
 L Device:R R12
 U 1 1 60985878
-P 7950 2050
-F 0 "R12" V 7750 2050 50  0000 C CNN
-F 1 "200" V 7850 2050 50  0000 C CNN
-F 2 "Resistor_SMD:R_0603_1608Metric" V 7880 2050 50  0001 C CNN
-F 3 "~" H 7950 2050 50  0001 C CNN
-	1    7950 2050
+P 4800 5000
+F 0 "R12" V 4600 5000 50  0000 C CNN
+F 1 "200" V 4700 5000 50  0000 C CNN
+F 2 "Resistor_SMD:R_0603_1608Metric" V 4730 5000 50  0001 C CNN
+F 3 "~" H 4800 5000 50  0001 C CNN
+	1    4800 5000
 	0    1    1    0
 $EndComp
@@
 L SC-STM32L412K8-rescue:Conn-My_Library-SC-STM32L412K8-rescue-SC-STM32L412K8-rescue-SC-STM32L412K8-rescue J10
 U 1 1 6098637F
-P 8200 2050
-F 0 "J10" H 8142 1825 50  0001 C CNN
-F 1 "Buzzer" H 8200 2150 50  0000 C CNN
-F 2 "My-library:SMD-CONN" H 8200 2050 50  0001 C CNN
-F 3 "~" H 8200 2050 50  0001 C CNN
-	1    8200 2050
+P 5050 5000
+F 0 "J10" H 4992 4775 50  0001 C CNN
+F 1 "Buzzer" H 5050 5100 50  0000 C CNN
+F 2 "My-library:SMD-CONN" H 5050 5000 50  0001 C CNN
+F 3 "~" H 5050 5000 50  0001 C CNN
+	1    5050 5000
 	1    0    0    -1
 $EndComp
@@
 L Transistor_FET:2N7002 Q1
 U 1 1 609A9FBA
-P 7700 1400
-F 0 "Q1" H 7906 1446 50  0000 L CNN
-F 1 "IRLML6344" H 7906 1355 50  0000 L CNN
-F 2 "Package_TO_SOT_SMD:SOT-23" H 7900 1325 50  0001 L CIN
-F 3 "https://www.fairchildsemi.com/datasheets/2N/2N7002.pdf" H 7700 1400 50  0001 L CNN
-	1    7700 1400
-	1    0    0    -1
-$EndComp
-Wire Wire Line
-	7800 1600 7800 1700
-Wire Wire Line
-	7500 1700 7800 1700
-Connection ~ 7800 1700
-Wire Wire Line
-	7350 1400 7500 1400
-Connection ~ 7500 1400
+P 4550 4350
+F 0 "Q1" H 4756 4396 50  0000 L CNN
+F 1 "IRLML6344" H 4756 4305 50  0000 L CNN
+F 2 "Package_TO_SOT_SMD:SOT-23" H 4750 4275 50  0001 L CIN
+F 3 "https://www.fairchildsemi.com/datasheets/2N/2N7002.pdf" H 4550 4350 50  0001 L CNN
+	1    4550 4350
+	1    0    0    -1
+$EndComp
+Wire Wire Line
+	4650 4550 4650 4650
+Wire Wire Line
+	4350 4650 4650 4650
+Connection ~ 4650 4650
+Wire Wire Line
+	4200 4350 4350 4350
+Connection ~ 4350 4350
 $Comp
 L Transistor_FET:2N7002 Q2
 U 1 1 609E193B
-P 7700 2250
-F 0 "Q2" H 7906 2296 50  0000 L CNN
-F 1 "IRLML6344" H 7906 2205 50  0000 L CNN
-F 2 "Package_TO_SOT_SMD:SOT-23" H 7900 2175 50  0001 L CIN
-F 3 "https://www.fairchildsemi.com/datasheets/2N/2N7002.pdf" H 7700 2250 50  0001 L CNN
-	1    7700 2250
-	1    0    0    -1
-$EndComp
-Wire Wire Line
-	7350 2250 7500 2250
-Connection ~ 7500 2250
-Wire Wire Line
-	7500 2550 7800 2550
-Wire Wire Line
-	7800 2550 7800 2450
-Connection ~ 7800 2550
+P 4550 5200
+F 0 "Q2" H 4756 5246 50  0000 L CNN
+F 1 "IRLML6344" H 4756 5155 50  0000 L CNN
+F 2 "Package_TO_SOT_SMD:SOT-23" H 4750 5125 50  0001 L CIN
+F 3 "https://www.fairchildsemi.com/datasheets/2N/2N7002.pdf" H 4550 5200 50  0001 L CNN
+	1    4550 5200
+	1    0    0    -1
+$EndComp
+Wire Wire Line
+	4200 5200 4350 5200
+Connection ~ 4350 5200
+Wire Wire Line
+	4350 5500 4650 5500
+Wire Wire Line
+	4650 5500 4650 5400
+Connection ~ 4650 5500
 Wire Wire Line
 	5950 3850 6150 3850
@@
 Wire Wire Line
 	4500 3000 4650 3000
+$Comp
+L My_Library:LTC1661CMS8 D3
+U 1 1 60B43F1F
+P 7250 1900
+F 0 "D3" H 7250 2315 50  0000 C CNN
+F 1 "LTC1662CMS8" H 7250 2224 50  0000 C CNN
+F 2 "Package_SO:MSOP-8_3x3mm_P0.65mm" H 7250 2300 50  0001 C CNN
+F 3 "" H 7250 1750 50  0001 C CNN
+	1    7250 1900
+	1    0    0    -1
+$EndComp
+$Comp
+L power:GND #PWR0103
+U 1 1 60B4B638
+P 7650 1850
+F 0 "#PWR0103" H 7650 1600 50  0001 C CNN
+F 1 "GND" H 7655 1677 50  0001 C CNN
+F 2 "" H 7650 1850 50  0001 C CNN
+F 3 "" H 7650 1850 50  0001 C CNN
+	1    7650 1850
+	0    -1   -1   0
+$EndComp
+$Comp
+L power:+3.3V #PWR0106
+U 1 1 60B51D5A
+P 7300 2800
+F 0 "#PWR0106" H 7300 2650 50  0001 C CNN
+F 1 "+3.3V" H 7315 2973 50  0000 C CNN
+F 2 "" H 7300 2800 50  0001 C CNN
+F 3 "" H 7300 2800 50  0001 C CNN
+	1    7300 2800
+	1    0    0    -1
+$EndComp
+Connection ~ 7300 2800
+$Comp
+L power:+3.3V #PWR0107
+U 1 1 60B52F4B
+P 7800 1950
+F 0 "#PWR0107" H 7800 1800 50  0001 C CNN
+F 1 "+3.3V" V 7700 2000 50  0000 L CNN
+F 2 "" H 7800 1950 50  0001 C CNN
+F 3 "" H 7800 1950 50  0001 C CNN
+	1    7800 1950
+	0    1    1    0
+$EndComp
+Text GLabel 4900 2200 0    50   Input ~ 0
+Adjust
+$Comp
+L Device:R R17
+U 1 1 60B5AD62
+P 8000 2050
+F 0 "R17" V 7900 2050 50  0000 C CNN
+F 1 "X" V 7800 2050 50  0000 C CNN
+F 2 "Resistor_SMD:R_0603_1608Metric" V 7930 2050 50  0001 C CNN
+F 3 "~" H 8000 2050 50  0001 C CNN
+	1    8000 2050
+	0    -1   -1   0
+$EndComp
+Text GLabel 8150 2050 2    50   Input ~ 0
+Adjust
+Wire Wire Line
+	4900 2200 5000 2200
+Connection ~ 5000 2200
+Wire Wire Line
+	7650 1950 7750 1950
+Wire Wire Line
+	6850 2050 6850 2300
+Wire Wire Line
+	6850 2300 7750 2300
+Wire Wire Line
+	7750 2300 7750 1950
+Connection ~ 7750 1950
+Wire Wire Line
+	7750 1950 7800 1950
+Wire Wire Line
+	7850 2050 7650 2050
+Text GLabel 6850 1950 0    50   Input ~ 0
+DI
+Text GLabel 6850 4750 0    50   Input ~ 0
+DI
+Text GLabel 6850 1850 0    50   Input ~ 0
+SC
+Text GLabel 7950 4500 2    50   Input ~ 0
+SC
+Text GLabel 6850 1750 0    50   Input ~ 0
+CS
+Text GLabel 6850 5150 0    50   Input ~ 0
+CS
 $EndSCHEMATC
