File: SC-STM32L412K8-light/SC-STM32L412K8.sch (KiCad schematic (older format))
At the start: 66 parts, among them J1 usb, J10 Buzzer, J11 Vibro, J12 +3v, J13 +vibro, J2 +29.6 SiPM, J3 TxD (20), J4 RxD (19), J5 SWDIO, J6 SWCLK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

Commit message: modified:   AndroidDoZer/app/release/app-release.apk 	modified:   AndroidDoZer/app/src/main/java/ru/starline/dozer/FullscreenActivity.java 	modified:   SC-STM32L412K8-light/SC-STM32L412K8-cache.lib 	modified:   SC-STM32L412K8-light/SC-STM32L412K8-rescue.lib 	modified:   SC-STM32L412K8-light/SC-STM32L412K8.sch 	modified:   SC-STM32L412K8-light/SC-STM32L412K8.sch-bak
Parts:
- D3: symbol My_Library:LTC1661CMS8 -> SC-STM32L412K8-rescue:LTC1661CMS8-My_Library
- R10: value 3k* -> 100
- R17: value X -> 10M
- R3: value 430k -> 432k
Other:
- moved on the sheet: D3, R17
Changed lines of the file:
@@
 P 5000 2000
 F 0 "R3" H 4800 2050 50  0000 L CNN
-F 1 "430k" H 4750 1950 50  0000 L CNN
+F 1 "432k" H 4750 1950 50  0000 L CNN
 F 2 "Resistor_SMD:R_0603_1608Metric" V 4930 2000 50  0001 C CNN
 F 3 "~" H 5000 2000 50  0001 C CNN
@@
 P 6500 1300
 F 0 "J2" H 6442 1075 50  0001 C CNN
-F 1 "+29.6 SiPM" H 6650 1200 50  0000 C CNN
+F 1 "+29.6 SiPM" H 6600 1400 50  0000 C CNN
 F 2 "My-library:SMD-CONN" H 6500 1300 50  0001 C CNN
 F 3 "~" H 6500 1300 50  0001 C CNN
@@
 P 5000 2350
 F 0 "R10" H 4750 2400 50  0000 L CNN
-F 1 "3k*" H 4800 2300 50  0000 L CNN
+F 1 "100" H 4800 2300 50  0000 L CNN
 F 2 "Resistor_SMD:R_0603_1608Metric" V 4930 2350 50  0001 C CNN
 F 3 "~" H 5000 2350 50  0001 C CNN
@@
 	4500 3000 4650 3000
 $Comp
-L My_Library:LTC1661CMS8 D3
+L SC-STM32L412K8-rescue:LTC1661CMS8-My_Library D3
 U 1 1 60B43F1F
-P 7250 1900
-F 0 "D3" H 7250 2315 50  0000 C CNN
-F 1 "LTC1662CMS8" H 7250 2224 50  0000 C CNN
-F 2 "Package_SO:MSOP-8_3x3mm_P0.65mm" H 7250 2300 50  0001 C CNN
-F 3 "" H 7250 1750 50  0001 C CNN
-	1    7250 1900
+P 7100 1750
+F 0 "D3" H 7100 2165 50  0000 C CNN
+F 1 "LTC1662CMS8" H 7100 2074 50  0000 C CNN
+F 2 "Package_SO:MSOP-8_3x3mm_P0.65mm" H 7100 2150 50  0001 C CNN
+F 3 "" H 7100 1600 50  0001 C CNN
+	1    7100 1750
 	1    0    0    -1
 $EndComp
@@
 L power:GND #PWR0103
 U 1 1 60B4B638
-P 7650 1850
-F 0 "#PWR0103" H 7650 1600 50  0001 C CNN
-F 1 "GND" H 7655 1677 50  0001 C CNN
-F 2 "" H 7650 1850 50  0001 C CNN
-F 3 "" H 7650 1850 50  0001 C CNN
-	1    7650 1850
+P 7500 1700
+F 0 "#PWR0103" H 7500 1450 50  0001 C CNN
+F 1 "GND" H 7505 1527 50  0001 C CNN
+F 2 "" H 7500 1700 50  0001 C CNN
+F 3 "" H 7500 1700 50  0001 C CNN
+	1    7500 1700
 	0    -1   -1   0
 $EndComp
@@
 L power:+3.3V #PWR0107
 U 1 1 60B52F4B
-P 7800 1950
-F 0 "#PWR0107" H 7800 1800 50  0001 C CNN
-F 1 "+3.3V" V 7700 2000 50  0000 L CNN
-F 2 "" H 7800 1950 50  0001 C CNN
-F 3 "" H 7800 1950 50  0001 C CNN
-	1    7800 1950
+P 7650 1800
+F 0 "#PWR0107" H 7650 1650 50  0001 C CNN
+F 1 "+3.3V" V 7550 1850 50  0000 L CNN
+F 2 "" H 7650 1800 50  0001 C CNN
+F 3 "" H 7650 1800 50  0001 C CNN
+	1    7650 1800
 	0    1    1    0
 $EndComp
@@
 L Device:R R17
 U 1 1 60B5AD62
-P 8000 2050
-F 0 "R17" V 7900 2050 50  0000 C CNN
-F 1 "X" V 7800 2050 50  0000 C CNN
-F 2 "Resistor_SMD:R_0603_1608Metric" V 7930 2050 50  0001 C CNN
-F 3 "~" H 8000 2050 50  0001 C CNN
-	1    8000 2050
+P 7850 1900
+F 0 "R17" V 7750 1900 50  0000 C CNN
+F 1 "10M" V 7650 1900 50  0000 C CNN
+F 2 "Resistor_SMD:R_0603_1608Metric" V 7780 1900 50  0001 C CNN
+F 3 "~" H 7850 1900 50  0001 C CNN
+	1    7850 1900
 	0    -1   -1   0
 $EndComp
-Text GLabel 8150 2050 2    50   Input ~ 0
+Text GLabel 8000 1900 2    50   Input ~ 0
 Adjust
 Wire Wire Line
@@
 Connection ~ 5000 2200
 Wire Wire Line
-	7650 1950 7750 1950
-Wire Wire Line
-	6850 2050 6850 2300
-Wire Wire Line
-	6850 2300 7750 2300
-Wire Wire Line
-	7750 2300 7750 1950
-Connection ~ 7750 1950
-Wire Wire Line
-	7750 1950 7800 1950
-Wire Wire Line
-	7850 2050 7650 2050
-Text GLabel 6850 1950 0    50   Input ~ 0
+	7500 1800 7600 1800
+Wire Wire Line
+	6700 1900 6700 2150
+Wire Wire Line
+	6700 2150 7600 2150
+Wire Wire Line
+	7600 2150 7600 1800
+Connection ~ 7600 1800
+Wire Wire Line
+	7600 1800 7650 1800
+Wire Wire Line
+	7700 1900 7500 1900
+Text GLabel 6700 1800 0    50   Input ~ 0
 DI
 Text GLabel 6850 4750 0    50   Input ~ 0
 DI
-Text GLabel 6850 1850 0    50   Input ~ 0
+Text GLabel 6700 1700 0    50   Input ~ 0
 SC
 Text GLabel 7950 4500 2    50   Input ~ 0
 SC
-Text GLabel 6850 1750 0    50   Input ~ 0
+Text GLabel 6700 1600 0    50   Input ~ 0
 CS
 Text GLabel 6850 5150 0    50   Input ~ 0
