File: kiCAD/SC-STM32L412K8-light/SC-STM32L412K8.kicad_pcb (KiCad board)
At the start: 2 copper layers, 31.6 x 15.1 mm, 66 parts, among them J1 usb, J10 Buzzer, J11 Vibro, J12 +3v, J13 +vibro, J2 +29.6 SiPM, J3 TxD (20), J4 RxD (19), J5 SWDIO, J6 SWCLK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

Commit message: modified:   kiCAD/SC-STM32L412K8-light/SC-STM32L412K8.kicad_pcb 	modified:   kiCAD/SC-STM32L412K8-light/SC-STM32L412K8.kicad_pcb-bak 	modified:   stm32Cube/STM32Code/.mxproject 	modified:   stm32Cube/STM32Code/.settings/language.settings.xml 	modified:   stm32Cube/STM32Code/Core/Src/main.c 	modified:   stm32Cube/STM32Code/SC4-LCD128x32.ioc 	modified:   stm32Cube/STM32L412K8code/.mxproject 	modified:   stm32Cube/STM32L412K8code/.settings/language.settings.xml 	modified:   stm32Cube/STM32L412K8code/STM32L412K8.ioc
Parts:
- moved C19 4.09 mm to (54.3, 63.3), turned to 90 degrees
- moved R2 0.14 mm to (56.1, 65.6)
- moved C3 0.10 mm to (37.7, 61.4)
Routing:
- net GND: track 198.3 -> 208.9 mm
- net +3V3: track 38.4 -> 41.0 mm
- net +BATT: track 50.5 -> 51.7 mm
- net Net-(C13-Pad1): track 13.2 -> 12.5 mm

Commit message: modified:   kiCAD/SC-STM32L412K8-light/SC-STM32L412K8.kicad_pcb 	modified:   kiCAD/SC-STM32L412K8-light/SC-STM32L412K8.kicad_pcb-bak
Parts:
- moved J3 0.28 mm to (53.6, 65.5)
- moved J4 0.28 mm to (53.6, 63.6)
- moved R17 0.22 mm to (43.2, 62.7)
- moved R3 0.19 mm to (43.2, 61.3)
Routing:
- net GND: track 208.9 -> 212.6 mm

Commit message: modified:   kiCAD/SC-STM32L412K8-light/SC-STM32L412K8.kicad_pcb 	modified:   kiCAD/SC-STM32L412K8-light/SC-STM32L412K8.kicad_pcb-bak 	modified:   kiCAD/SC-STM32L412K8-light/SC-STM32L412K8.sch 	modified:   kiCAD/SC-STM32L412K8-light/SC-STM32L412K8.sch-bak
Parts:
- moved C11 0.22 mm to (49.9, 57.2)
- moved C14 0.22 mm to (51.7, 57.2)
- moved C2 0.08 mm to (54.3, 59.9)

Commit message: modified:   kiCAD/SC-STM32L412K8-light/SC-STM32L412K8.kicad_pcb 	modified:   kiCAD/SC-STM32L412K8-light/SC-STM32L412K8.kicad_pcb-bak 	modified:   kiCAD/SC-STM32L412K8-light/SC-STM32L412K8.sch 	modified:   kiCAD/SC-STM32L412K8-light/SC-STM32L412K8.sch-bak
Parts:
- added J14: gndBT, My-library:SMD-CONN, F.Cu at (32.2, 65.3)
- added J15: -BAT, My-library:SMD-CONN, F.Cu at (40.1, 65.7)
- L1: value LQM21FN100N -> L1 LQM21FN100N
- L2: value LQH31MN220J03L -> L2 LQH31MN220J03L
- L3: value MLZ2012M470WT000 -> L3 MLZ2012M470WT000
- L4: value MLZ2012M470WT000 -> L4 MLZ2012M470WT000
- Q1, Q2: value IRLML6344 -> IRLML0060RTPbF
- R10: value 3k* -> 442k
- R17: value 100k -> 30M
- R3: value 430k -> 4.7k

Commit message: modified:   kiCAD/SC-STM32L412K8-light/SC-STM32L412K8.kicad_pcb 	modified:   kiCAD/SC-STM32L412K8-light/SC-STM32L412K8.kicad_pcb-bak 	modified:   stm32Cube/STM32L412K8code/.settings/language.settings.xml
Parts:
- moved C19 0.46 mm to (54.3, 63.7)
Routing:
- net +3V3: track 40.9 -> 40.1 mm

Commit message: изменено:      kiCAD/SC-STM32L412K8-light/SC-STM32L412K8.kicad_pcb 	изменено:      kiCAD/SC-STM32L412K8-light/SC-STM32L412K8.kicad_pcb-bak
Parts:
- R17: value 30M -> 10M

Commit message: изменено:      kiCAD/SC-STM32L412K8-light/SC-STM32L412K8.kicad_pcb 	изменено:      kiCAD/SC-STM32L412K8-light/SC-STM32L412K8.kicad_pcb-bak 	изменено:      kiCAD/SC-STM32L412K8-light/SC-STM32L412K8.sch 	изменено:      kiCAD/SC-STM32L412K8-light/SC-STM32L412K8.sch-bak 	изменено:      kiCAD/SC-STM32L412K8-light/bom/ibom.html.gz
Parts:
- C1, C12, C13, C15, C16, C17, C18, C19, C2, C3, C4: value 22uF -> GRM21BR60J226M
- C11, C14, C6, C7, C8: value C3216X7R1H106K160AC -> GRM21BC8YA106KE11L

Commit message: изменено:      Documents/isotops.list 	изменено:      kiCAD/SC-STM32L412K8-light/SC-STM32L412K8.kicad_pcb
Parts:
- D2: value MBR0540 -> BAT46ZFILM
