File: kiCAD/SC-STM32L412K8-light/SC-STM32L412K8.kicad_pcb (KiCad board)
At the start: 2 copper layers, 31.6 x 15.1 mm, 68 parts, among them J1 usb, J10 Buzzer, J11 Vibro, J12 +3v, J13 +vibro, J14 gndBT, J15 -BAT, J2 +29.6 SiPM, J3 TxD (20), J4 RxD (19)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

Commit message: изменено:      kiCAD/SC-STM32L412K8-light/SC-STM32L412K8.kicad_pcb 	изменено:      kiCAD/SC-STM32L412K8-light/SC-STM32L412K8.kicad_pcb-bak 	изменено:      kiCAD/SC-STM32L412K8-light/SC-STM32L412K8.sch 	изменено:      kiCAD/SC-STM32L412K8-light/SC-STM32L412K8.sch-bak 	новый файл:    picture/IMG_20211115_132411.jpg
Parts:
- moved C5 0.61 mm to (42.1, 59.2)
- moved R5 0.57 mm to (43.5, 59.2)
- moved C7 0.10 mm to (42.7, 56.8)
Routing:
- net GND: track 212.6 -> 214.3 mm

Commit message: изменено:      kiCAD/SC-STM32L412K8-light/SC-STM32L412K8.kicad_pcb 	изменено:      kiCAD/SC-STM32L412K8-light/SC-STM32L412K8.kicad_pcb-bak
Parts:
- moved J13 0.82 mm to (32.1, 54.0)

Commit message: изменено:      kiCAD/SC-STM32L412K8-light/SC-STM32L412K8-cache.lib 	изменено:      kiCAD/SC-STM32L412K8-light/SC-STM32L412K8-rescue.lib 	изменено:      kiCAD/SC-STM32L412K8-light/SC-STM32L412K8.kicad_pcb 	изменено:      kiCAD/SC-STM32L412K8-light/SC-STM32L412K8.kicad_pcb-bak 	изменено:      kiCAD/SC-STM32L412K8-light/SC-STM32L412K8.sch 	изменено:      kiCAD/SC-STM32L412K8-light/SC-STM32L412K8.sch-bak 	изменено:      kiCAD/SC-STM32L412K8-light/fp-info-cache 	изменено:      stm32Cube/STM32L412K8code/Debug/Core/Src/main.o 	изменено:      stm32Cube/STM32L412K8code/Debug/Core/Src/stm32l4xx_hal_msp.o 	изменено:      stm32Cube/STM32L412K8code/Debug/Core/Src/stm32l4xx_it.o 	изменено:      stm32Cube/STM32L412K8code/Debug/Core/Src/syscalls.o 	изменено:      stm32Cube/STM32L412K8code/Debug/Core/Src/sysmem.o 	изменено:      stm32Cube/STM32L412K8code/Debug/Core/Src/system_stm32l4xx.o 	изменено:      stm32Cube/STM32L412K8code/Debug/Core/Startup/startup_stm32l412k8tx.o 	изменено:      stm32Cube/STM32L412K8code/Debug/Drivers/STM32L4xx_HAL_Driver/Src/stm32l4xx_hal.o 	изменено:      stm32Cube/STM32L412K8code/Debug/Drivers/STM32L4xx_HAL_Driver/Src/stm32l4xx_hal_adc.o 	изменено:      stm32Cube/STM32L412K8code/Debug/Drivers/STM32L4xx_HAL_Driver/Src/stm32l4xx_hal_adc_ex.o 	изменено:      stm32Cube/STM32L412K8code/Debug/Drivers/STM32L4xx_HAL_Driver/Src/stm32l4xx_hal_cortex.o 	изменено:      stm32Cube/STM32L412K8code/Debug/Drivers/STM32L4xx_HAL_Driver/Src/stm32l4xx_hal_dma.o 	изменено:      stm32Cube/STM32L412K8code/Debug/Drivers/STM32L4xx_HAL_Driver/Src/stm32l4xx_hal_dma_ex.o 	изменено:      stm32Cube/STM32L412K8code/Debug/Drivers/STM32L4xx_HAL_Driver/Src/stm32l4xx_hal_exti.o 	изменено:      stm32Cube/STM32L412K8code/Debug/Drivers/STM32L4xx_HAL_Driver/Src/stm32l4xx_hal_flash.o 	изменено:      stm32Cube/STM32L412K8code/Debug/Drivers/STM32L4xx_HAL_Driver/Src/stm32l4xx_hal_flash_ex.o 	изменено:      stm32Cube/STM32L412K8code/Debug/Drivers/STM32L4xx_HAL_Driver/Src/stm32l4xx_hal_flash_ramfunc.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
Parts:
- removed J10: Buzzer, My-library:SMD-CONN
- removed R12: 200, Resistor_SMD:R_0603_1608Metric
- added BZ1: Buzzer, My-library:BuzerSMD, B.Cu at (36.5, 65.1)
- C1, C13, C15, C16, C17, C19, C2, C3, C4: footprint Capacitor_SMD:C_0805_2012Metric -> Capacitor_SMD:C_0603_1608Metric
- D1, D7: footprint LED_SMD:LED_0805_2012Metric -> LED_SMD:LED_0603_1608Metric
- R10, R17, R3: footprint Resistor_SMD:R_0603_1608Metric -> Resistor_SMD:R_0402_1005Metric
- moved J11 1.98 mm to (36.6, 65.3)
- moved Q2 1.37 mm to (41.5, 65.7)
- moved R17 0.71 mm to (42.7, 62.2)
- moved R3 0.56 mm to (42.7, 61.2)
- moved C17 0.29 mm to (42.4, 56.0)
- moved C15 0.27 mm to (57.3, 57.4)
- moved C19 0.23 mm to (54.3, 64.0)
- moved C1 0.22 mm to (34.5, 57.4)
- moved C13 0.21 mm to (34.6, 60.8)
- moved C2 0.21 mm to (54.1, 59.8)
- moved R10 0.18 mm to (40.7, 61.2)
- moved C3 0.18 mm to (37.5, 61.4)
- moved C16 0.17 mm to (50.9, 65.5)
Routing:
- net +BATT: track 51.3 -> 67.3 mm
- net Net-(J11-Pad1): track 2.15 -> 0.13 mm
- net Net-(J10-Pad1): track 1.83 -> 0.00 mm
- net Buzer: track 4.40 -> 3.45 mm
- net GND: track 214.3 -> 213.3 mm, vias 10 -> 11
- net Net-(BZ1-Pad2): track 1.13 -> 2.02 mm
- net Net-(D3-Pad5): track 2.86 -> 3.69 mm

Commit message: изменено:      kiCAD/SC-STM32L412K8-light/SC-STM32L412K8.kicad_pcb 	изменено:      kiCAD/SC-STM32L412K8-light/SC-STM32L412K8.kicad_pcb-bak 	изменено:      kiCAD/SC-STM32L412K8-light/SC-STM32L412K8.sch 	изменено:      kiCAD/SC-STM32L412K8-light/SC-STM32L412K8.sch-bak
Parts:
- C1, C13, C15, C16, C17, C19, C2, C3, C4: value GRM21BR60J226M -> 1uF

Commit message: изменено:      Release/all.zip 	изменено:      kiCAD/SC-STM32L412K8-light/SC-STM32L412K8.kicad_pcb 	изменено:      kiCAD/SC-STM32L412K8-light/SC-STM32L412K8.kicad_pcb-bak
Parts:
- moved J11 3.62 mm to (39.4, 63.0)
- moved BZ1 1.05 mm to (35.5, 65.2)
Routing:
- net GND: track 213.3 -> 221.6 mm
- net Net-(J11-Pad1): track 0.13 -> 5.37 mm
- net Net-(BZ1-Pad2): track 2.02 -> 3.06 mm
- net +BATT: track 67.3 -> 66.5 mm
