File: kiCAD/SC-STM32L412K8-light/SC-STM32L412K8.sch (KiCad schematic (older format))
At the start: 68 parts, among them J1 usb, J10 Buzzer, J11 Vibro, J12 +3v, J13 +vibro, J14 gndBT, J15 -BAT, J2 +29.6 SiPM, J3 TxD (20), J4 RxD (19)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

Commit message: изменено:      kiCAD/SC-STM32L412K8-light/SC-STM32L412K8.kicad_pcb 	изменено:      kiCAD/SC-STM32L412K8-light/SC-STM32L412K8.kicad_pcb-bak 	изменено:      kiCAD/SC-STM32L412K8-light/SC-STM32L412K8.sch 	изменено:      kiCAD/SC-STM32L412K8-light/SC-STM32L412K8.sch-bak 	новый файл:    picture/IMG_20211115_132411.jpg
Connections:
- no-connect marks 0 -> 10
Changed lines of the file:
@@
 	1    0    0    -1
 $EndComp
+NoConn ~ 7950 4200
+NoConn ~ 7950 4600
+NoConn ~ 7950 4700
+NoConn ~ 7950 4800
+NoConn ~ 7950 4950
+NoConn ~ 7950 5050
+NoConn ~ 6850 4450
+NoConn ~ 6850 4350
+NoConn ~ 6850 4150
+NoConn ~ 6850 3950
 $EndSCHEMATC

Commit message: изменено:      kiCAD/SC-STM32L412K8-light/SC-STM32L412K8-cache.lib 	изменено:      kiCAD/SC-STM32L412K8-light/SC-STM32L412K8-rescue.lib 	изменено:      kiCAD/SC-STM32L412K8-light/SC-STM32L412K8.kicad_pcb 	изменено:      kiCAD/SC-STM32L412K8-light/SC-STM32L412K8.kicad_pcb-bak 	изменено:      kiCAD/SC-STM32L412K8-light/SC-STM32L412K8.sch 	изменено:      kiCAD/SC-STM32L412K8-light/SC-STM32L412K8.sch-bak 	изменено:      kiCAD/SC-STM32L412K8-light/fp-info-cache 	изменено:      stm32Cube/STM32L412K8code/Debug/Core/Src/main.o 	изменено:      stm32Cube/STM32L412K8code/Debug/Core/Src/stm32l4xx_hal_msp.o 	изменено:      stm32Cube/STM32L412K8code/Debug/Core/Src/stm32l4xx_it.o 	изменено:      stm32Cube/STM32L412K8code/Debug/Core/Src/syscalls.o 	изменено:      stm32Cube/STM32L412K8code/Debug/Core/Src/sysmem.o 	изменено:      stm32Cube/STM32L412K8code/Debug/Core/Src/system_stm32l4xx.o 	изменено:      stm32Cube/STM32L412K8code/Debug/Core/Startup/startup_stm32l412k8tx.o 	изменено:      stm32Cube/STM32L412K8code/Debug/Drivers/STM32L4xx_HAL_Driver/Src/stm32l4xx_hal.o 	изменено:      stm32Cube/STM32L412K8code/Debug/Drivers/STM32L4xx_HAL_Driver/Src/stm32l4xx_hal_adc.o 	изменено:      stm32Cube/STM32L412K8code/Debug/Drivers/STM32L4xx_HAL_Driver/Src/stm32l4xx_hal_adc_ex.o 	изменено:      stm32Cube/STM32L412K8code/Debug/Drivers/STM32L4xx_HAL_Driver/Src/stm32l4xx_hal_cortex.o 	изменено:      stm32Cube/STM32L412K8code/Debug/Drivers/STM32L4xx_HAL_Driver/Src/stm32l4xx_hal_dma.o 	изменено:      stm32Cube/STM32L412K8code/Debug/Drivers/STM32L4xx_HAL_Driver/Src/stm32l4xx_hal_dma_ex.o 	изменено:      stm32Cube/STM32L412K8code/Debug/Drivers/STM32L4xx_HAL_Driver/Src/stm32l4xx_hal_exti.o 	изменено:      stm32Cube/STM32L412K8code/Debug/Drivers/STM32L4xx_HAL_Driver/Src/stm32l4xx_hal_flash.o 	изменено:      stm32Cube/STM32L412K8code/Debug/Drivers/STM32L4xx_HAL_Driver/Src/stm32l4xx_hal_flash_ex.o 	изменено:      stm32Cube/STM32L412K8code/Debug/Drivers/STM32L4xx_HAL_Driver/Src/stm32l4xx_hal_flash_ramfunc.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
Parts:
- removed J10: Buzzer, My-library:SMD-CONN, symbol SC-STM32L412K8-rescue:Conn-My_Library-SC-STM32L412K8-rescue-SC-STM32L412K8-resc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
- removed R12: 200, Resistor_SMD:R_0603_1608Metric, symbol Device:R
- added BZ1: Buzzer, My-library:BuzerSMD, symbol Device:Buzzer
- C1, C13, C15, C16, C17, C19, C2, C3, C4: footprint Capacitor_SMD:C_0805_2012Metric -> Capacitor_SMD:C_0603_1608Metric
- D1, D7: footprint LED_SMD:LED_0805_2012Metric -> LED_SMD:LED_0603_1608Metric
- J1: symbol Connector:USB_B_Micro -> SC-STM32L412K8-rescue:USB_B_Micro-Connector
- R10, R17, R3: footprint Resistor_SMD:R_0603_1608Metric -> Resistor_SMD:R_0402_1005Metric
Other:
- moved on the sheet: Q1, R16
Changed lines of the file:
@@
 F 0 "R3" H 4800 2050 50  0000 L CNN
 F 1 "4.7k" H 4750 1950 50  0000 L CNN
-F 2 "Resistor_SMD:R_0603_1608Metric" V 4930 2000 50  0001 C CNN
+F 2 "Resistor_SMD:R_0402_1005Metric" V 4930 2000 50  0001 C CNN
 F 3 "~" H 5000 2000 50  0001 C CNN
 	1    5000 2000
@@
 F 0 "C17" H 7050 3900 50  0000 L CNN
 F 1 "GRM21BR60J226M" H 7050 3800 50  0001 L CNN
-F 2 "Capacitor_SMD:C_0805_2012Metric" H 7188 3400 50  0001 C CNN
+F 2 "Capacitor_SMD:C_0603_1608Metric" H 7188 3400 50  0001 C CNN
 F 3 "~" H 7150 3550 50  0001 C CNN
 	1    7150 3550
@@
 F 0 "C16" H 6800 3900 50  0000 L CNN
 F 1 "GRM21BR60J226M" H 6800 3800 50  0001 L CNN
-F 2 "Capacitor_SMD:C_0805_2012Metric" H 6988 3400 50  0001 C CNN
+F 2 "Capacitor_SMD:C_0603_1608Metric" H 6988 3400 50  0001 C CNN
 F 3 "~" H 6950 3550 50  0001 C CNN
 	1    6950 3550
@@
 F 0 "D1" V 4550 3150 50  0000 R CNN
 F 1 "LED" V 4450 3200 50  0000 R CNN
-F 2 "LED_SMD:LED_0805_2012Metric" H 4500 3250 50  0001 C CNN
+F 2 "LED_SMD:LED_0603_1608Metric" H 4500 3250 50  0001 C CNN
 F 3 "~" H 4500 3250 50  0001 C CNN
 	1    4500 3250
@@
 F 0 "C13" H 5350 3850 50  0000 L CNN
 F 1 "GRM21BR60J226M" H 5300 3650 50  0001 L CNN
-F 2 "Capacitor_SMD:C_0805_2012Metric" H 5588 3600 50  0001 C CNN
+F 2 "Capacitor_SMD:C_0603_1608Metric" H 5588 3600 50  0001 C CNN
 F 3 "~" H 5550 3750 50  0001 C CNN
 	1    5550 3750
@@
 $EndComp
 $Comp
-L Connector:USB_B_Micro J1
+L SC-STM32L412K8-rescue:USB_B_Micro-Connector J1
 U 1 1 603CD9A3
 P 4100 3050
@@
 F 0 "C3" H 4200 2300 50  0000 R CNN
 F 1 "GRM21BR60J226M" H 4200 2400 50  0001 R CNN
-F 2 "Capacitor_SMD:C_0805_2012Metric" H 4338 2200 50  0001 C CNN
+F 2 "Capacitor_SMD:C_0603_1608Metric" H 4338 2200 50  0001 C CNN
 F 3 "~" H 4300 2350 50  0001 C CNN
 	1    4300 2350
@@
 F 0 "C1" H 3850 2150 50  0000 R CNN
 F 1 "GRM21BR60J226M" H 3850 2250 50  0001 R CNN
-F 2 "Capacitor_SMD:C_0805_2012Metric" H 3938 2200 50  0001 C CNN
+F 2 "Capacitor_SMD:C_0603_1608Metric" H 3938 2200 50  0001 C CNN
 F 3 "GRM21BR60J226M" H 3900 2350 50  0001 C CNN
 	1    3900 2350
@@
 F 0 "C19" H 7400 3100 50  0000 L CNN
 F 1 "GRM21BR60J226M" H 7400 3000 50  0001 L CNN
-F 2 "Capacitor_SMD:C_0805_2012Metric" H 7088 2800 50  0001 C CNN
+F 2 "Capacitor_SMD:C_0603_1608Metric" H 7088 2800 50  0001 C CNN
 F 3 "~" H 7050 2950 50  0001 C CNN
 	1    7050 2950
@@
 F 0 "C15" H 6250 2750 50  0000 L CNN
 F 1 "GRM21BR60J226M" H 6250 2650 50  0001 L CNN
-F 2 "Capacitor_SMD:C_0805_2012Metric" H 6388 2800 50  0001 C CNN
+F 2 "Capacitor_SMD:C_0603_1608Metric" H 6388 2800 50  0001 C CNN
 F 3 "~" H 6350 2950 50  0001 C CNN
 	1    6350 2950
@@
 F 0 "D7" V 8300 4400 50  0000 R CNN
 F 1 "LED" V 8200 4400 50  0000 R CNN
-F 2 "LED_SMD:LED_0805_2012Metric" H 8250 4550 50  0001 C CNN
+F 2 "LED_SMD:LED_0603_1608Metric" H 8250 4550 50  0001 C CNN
 F 3 "~" H 8250 4550 50  0001 C CNN
 	1    8250 4550
@@
 L Device:R R16
 U 1 1 604FB12B
-P 4350 4500
-F 0 "R16" H 4500 4450 50  0000 C CNN
-F 1 "100k" H 4500 4550 50  0000 C CNN
-F 2 "Resistor_SMD:R_0603_1608Metric" V 4280 4500 50  0001 C CNN
-F 3 "~" H 4350 4500 50  0001 C CNN
-	1    4350 4500
+P 4350 4400
+F 0 "R16" H 4500 4350 50  0000 C CNN
+F 1 "100k" H 4500 4450 50  0000 C CNN
+F 2 "Resistor_SMD:R_0603_1608Metric" V 4280 4400 50  0001 C CNN
+F 3 "~" H 4350 4400 50  0001 C CNN
+	1    4350 4400
 	-1   0    0    1
 $EndComp
@@
 L power:GND #PWR0102
 U 1 1 604FC90E
-P 4650 4650
-F 0 "#PWR0102" H 4650 4400 50  0001 C CNN
-F 1 "GND" H 4655 4477 50  0001 C CNN
-F 2 "" H 4650 4650 50  0001 C CNN
-F 3 "" H 4650 4650 50  0001 C CNN
-	1    4650 4650
+P 4650 4550
+F 0 "#PWR0102" H 4650 4300 50  0001 C CNN
+F 1 "GND" H 4655 4377 50  0001 C CNN
+F 2 "" H 4650 4550 50  0001 C CNN
+F 3 "" H 4650 4550 50  0001 C CNN
+	1    4650 4550
 	1    0    0    -1
 $EndComp
@@
 L SC-STM32L412K8-rescue:Conn-My_Library-SC-STM32L412K8-rescue-SC-STM32L412K8-rescue-SC-STM32L412K8-rescue J11
 U 1 1 605058F1
-P 4750 4150
-F 0 "J11" H 4692 3925 50  0001 C CNN
-F 1 "Vibro" H 4750 4250 50  0000 C CNN
-F 2 "My-library:SMD-CONN" H 4750 4150 50  0001 C CNN
-F 3 "~" H 4750 4150 50  0001 C CNN
-	1    4750 4150
+P 4750 4050
+F 0 "J11" H 4692 3825 50  0001 C CNN
+F 1 "Vibro" H 4750 4150 50  0000 C CNN
+F 2 "My-library:SMD-CONN" H 4750 4050 50  0001 C CNN
+F 3 "~" H 4750 4050 50  0001 C CNN
+	1    4750 4050
 	1    0    0    -1
 $EndComp
@@
 F 0 "C2" H 5450 4550 50  0000 L CNN
 F 1 "GRM21BR60J226M" H 5400 4450 50  0001 L CNN
-F 2 "Capacitor_SMD:C_0805_2012Metric" H 5688 4500 50  0001 C CNN
+F 2 "Capacitor_SMD:C_0603_1608Metric" H 5688 4500 50  0001 C CNN
 F 3 "~" H 5650 4650 50  0001 C CNN
 	1    5650 4650
@@
 	0    -1   -1   0
 $EndComp
-Text GLabel 4200 4350 0    50   Input ~ 0
+Text GLabel 4200 4250 0    50   Input ~ 0
 Vibro
 Text GLabel 6850 4050 0    50   Input ~ 0
@@
 F 0 "C4" H 5400 2800 50  0000 R CNN
 F 1 "GRM21BR60J226M" H 5400 2900 50  0001 R CNN
-F 2 "Capacitor_SMD:C_0805_2012Metric" H 5488 2850 50  0001 C CNN
+F 2 "Capacitor_SMD:C_0603_1608Metric" H 5488 2850 50  0001 C CNN
 F 3 "~" H 5450 3000 50  0001 C CNN
 	1    5450 3000
@@
 F 0 "R10" H 4750 2400 50  0000 L CNN
 F 1 "442k" H 4750 2300 50  0000 L CNN
-F 2 "Resistor_SMD:R_0603_1608Metric" V 4930 2350 50  0001 C CNN
+F 2 "Resistor_SMD:R_0402_1005Metric" V 4930 2350 50  0001 C CNN
 F 3 "~" H 5000 2350 50  0001 C CNN
 	1    5000 2350
@@
 	5800 2200 5600 2200
 $Comp
-L Device:R R12
-U 1 1 60985878
-P 4800 5000
-F 0 "R12" V 4600 5000 50  0000 C CNN
-F 1 "200" V 4700 5000 50  0000 C CNN
-F 2 "Resistor_SMD:R_0603_1608Metric" V 4730 5000 50  0001 C CNN
-F 3 "~" H 4800 5000 50  0001 C CNN
-	1    4800 5000
-	0    1    1    0
-$EndComp
-$Comp
-L SC-STM32L412K8-rescue:Conn-My_Library-SC-STM32L412K8-rescue-SC-STM32L412K8-rescue-SC-STM32L412K8-rescue J10
-U 1 1 6098637F
-P 5050 5000
-F 0 "J10" H 4992 4775 50  0001 C CNN
-F 1 "Buzzer" H 5050 5100 50  0000 C CNN
-F 2 "My-library:SMD-CONN" H 5050 5000 50  0001 C CNN
-F 3 "~" H 5050 5000 50  0001 C CNN
-	1    5050 5000
-	1    0    0    -1
-$EndComp
-$Comp
 L Transistor_FET:2N7002 Q1
 U 1 1 609A9FBA
-P 4550 4350
-F 0 "Q1" H 4400 4600 50  0000 L CNN
-F 1 "IRLML0060RTPbF" H 3900 4500 50  0000 L CNN
-F 2 "Package_TO_SOT_SMD:SOT-23" H 4750 4275 50  0001 L CIN
-F 3 "https://www.fairchildsemi.com/datasheets/2N/2N7002.pdf" H 4550 4350 50  0001 L CNN
-	1    4550 4350
-	1    0    0    -1
-$EndComp
-Wire Wire Line
-	4650 4550 4650 4650
-Wire Wire Line
-	4350 4650 4650 4650
-Connection ~ 4650 4650
-Wire Wire Line
-	4200 4350 4350 4350
-Connection ~ 4350 4350
+P 4550 4250
+F 0 "Q1" H 4400 4500 50  0000 L CNN
+F 1 "IRLML0060RTPbF" H 3900 4400 50  0000 L CNN
+F 2 "Package_TO_SOT_SMD:SOT-23" H 4750 4175 50  0001 L CIN
+F 3 "https://www.fairchildsemi.com/datasheets/2N/2N7002.pdf" H 4550 4250 50  0001 L CNN
+	1    4550 4250
+	1    0    0    -1
+$EndComp
+Wire Wire Line
+	4650 4450 4650 4550
+Wire Wire Line
+	4350 4550 4650 4550
+Connection ~ 4650 4550
+Wire Wire Line
+	4200 4250 4350 4250
+Connection ~ 4350 4250
 $Comp
 L Transistor_FET:2N7002 Q2
@@
 F 0 "R17" V 7750 1900 50  0000 C CNN
 F 1 "10M" V 7650 1900 50  0000 C CNN
-F 2 "Resistor_SMD:R_0603_1608Metric" V 7780 1900 50  0001 C CNN
+F 2 "Resistor_SMD:R_0402_1005Metric" V 7780 1900 50  0001 C CNN
 F 3 "~" H 7850 1900 50  0001 C CNN
 	1    7850 1900
@@
 NoConn ~ 6850 4150
 NoConn ~ 6850 3950
+$Comp
+L Device:Buzzer BZ1
+U 1 1 6325DE2C
+P 4750 4900
+F 0 "BZ1" H 4902 4929 50  0000 L CNN
+F 1 "Buzzer" H 4902 4838 50  0000 L CNN
+F 2 "My-library:BuzerSMD" V 4725 5000 50  0001 C CNN
+F 3 "~" V 4725 5000 50  0001 C CNN
+	1    4750 4900
+	1    0    0    -1
+$EndComp
+$Comp
+L power:+BATT #PWR0110
+U 1 1 63278ED6
+P 4650 4800
+F 0 "#PWR0110" H 4650 4650 50  0001 C CNN
+F 1 "+BATT" V 4700 5000 50  0000 C CNN
+F 2 "" H 4650 4800 50  0001 C CNN
+F 3 "" H 4650 4800 50  0001 C CNN
+	1    4650 4800
+	0    -1   -1   0
+$EndComp
 $EndSCHEMATC

Commit message: изменено:      kiCAD/SC-STM32L412K8-light/SC-STM32L412K8.kicad_pcb 	изменено:      kiCAD/SC-STM32L412K8-light/SC-STM32L412K8.kicad_pcb-bak 	изменено:      kiCAD/SC-STM32L412K8-light/SC-STM32L412K8.sch 	изменено:      kiCAD/SC-STM32L412K8-light/SC-STM32L412K8.sch-bak
Parts:
- C1, C13, C15, C16, C17, C19, C2, C3, C4: value GRM21BR60J226M -> 1uF
Other:
- note removed: "C1, C2, C3, C4, C12, C13, C15, C16, C17, C18, C19 GRM21BR60J226M"
Changed lines of the file:
@@
 P 7150 3550
 F 0 "C17" H 7050 3900 50  0000 L CNN
-F 1 "GRM21BR60J226M" H 7050 3800 50  0001 L CNN
+F 1 "1uF" H 7050 3800 50  0001 L CNN
 F 2 "Capacitor_SMD:C_0603_1608Metric" H 7188 3400 50  0001 C CNN
 F 3 "~" H 7150 3550 50  0001 C CNN
@@
 P 6950 3550
 F 0 "C16" H 6800 3900 50  0000 L CNN
-F 1 "GRM21BR60J226M" H 6800 3800 50  0001 L CNN
+F 1 "1uF" H 6800 3800 50  0001 L CNN
 F 2 "Capacitor_SMD:C_0603_1608Metric" H 6988 3400 50  0001 C CNN
 F 3 "~" H 6950 3550 50  0001 C CNN
@@
 P 5550 3750
 F 0 "C13" H 5350 3850 50  0000 L CNN
-F 1 "GRM21BR60J226M" H 5300 3650 50  0001 L CNN
+F 1 "1uF" H 5300 3650 50  0001 L CNN
 F 2 "Capacitor_SMD:C_0603_1608Metric" H 5588 3600 50  0001 C CNN
 F 3 "~" H 5550 3750 50  0001 C CNN
@@
 P 4300 2350
 F 0 "C3" H 4200 2300 50  0000 R CNN
-F 1 "GRM21BR60J226M" H 4200 2400 50  0001 R CNN
+F 1 "1uF" H 4200 2400 50  0001 R CNN
 F 2 "Capacitor_SMD:C_0603_1608Metric" H 4338 2200 50  0001 C CNN
 F 3 "~" H 4300 2350 50  0001 C CNN
@@
 P 3900 2350
 F 0 "C1" H 3850 2150 50  0000 R CNN
-F 1 "GRM21BR60J226M" H 3850 2250 50  0001 R CNN
+F 1 "1uF" H 3850 2250 50  0001 R CNN
 F 2 "Capacitor_SMD:C_0603_1608Metric" H 3938 2200 50  0001 C CNN
 F 3 "GRM21BR60J226M" H 3900 2350 50  0001 C CNN
@@
 P 7050 2950
 F 0 "C19" H 7400 3100 50  0000 L CNN
-F 1 "GRM21BR60J226M" H 7400 3000 50  0001 L CNN
+F 1 "1uF" H 7400 3000 50  0001 L CNN
 F 2 "Capacitor_SMD:C_0603_1608Metric" H 7088 2800 50  0001 C CNN
 F 3 "~" H 7050 2950 50  0001 C CNN
@@
 P 6350 2950
 F 0 "C15" H 6250 2750 50  0000 L CNN
-F 1 "GRM21BR60J226M" H 6250 2650 50  0001 L CNN
+F 1 "1uF" H 6250 2650 50  0001 L CNN
 F 2 "Capacitor_SMD:C_0603_1608Metric" H 6388 2800 50  0001 C CNN
 F 3 "~" H 6350 2950 50  0001 C CNN
@@
 P 5650 4650
 F 0 "C2" H 5450 4550 50  0000 L CNN
-F 1 "GRM21BR60J226M" H 5400 4450 50  0001 L CNN
+F 1 "1uF" H 5400 4450 50  0001 L CNN
 F 2 "Capacitor_SMD:C_0603_1608Metric" H 5688 4500 50  0001 C CNN
 F 3 "~" H 5650 4650 50  0001 C CNN
@@
 P 5450 3000
 F 0 "C4" H 5400 2800 50  0000 R CNN
-F 1 "GRM21BR60J226M" H 5400 2900 50  0001 R CNN
+F 1 "1uF" H 5400 2900 50  0001 R CNN
 F 2 "Capacitor_SMD:C_0603_1608Metric" H 5488 2850 50  0001 C CNN
 F 3 "~" H 5450 3000 50  0001 C CNN
@@
 Wire Wire Line
 	4000 3450 4000 3650
-Text Notes 4150 850  0    50   ~ 0
-C1, C2, C3, C4, C12, C13, C15, C16, C17, C18, C19  GRM21BR60J226M
 Wire Wire Line
 	6350 4500 6350 3400
