File: kiCAD/SC-STM32L412K8-light_v2/SC-STM32L412K8.kicad_pcb (KiCad board)
At the start: 2 copper layers, 31.6 x 15.1 mm, 70 parts, among them J1 usb, J10 gnd, J11 Vibro, J12 +2.8v, J13 +vibro, J14 gndBT, J15 -BAT, J16 +2.8v, J2 +29.6 SiPM, J3 TxD(20)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

Commit message: удалено:       kiCAD/SC-STM32L412K8-light_v2/SC-STM32L412K8-backups/SC-STM32L412K8-2023-09-11_154928.zip 	изменено:      kiCAD/SC-STM32L412K8-light_v2/SC-STM32L412K8.kicad_pcb 	изменено:      kiCAD/SC-STM32L412K8-light_v2/SC-STM32L412K8.kicad_prl 	изменено:      kiCAD/SC-STM32L412K8-light_v2/SC-STM32L412K8.kicad_sch 	изменено:      kiCAD/SC-STM32L412K8-light_v2/fp-info-cache 	изменено:      kiCAD/SC-STM32L412K8-light_v2/gerber/Border.gbr 	изменено:      kiCAD/SC-STM32L412K8-light_v2/gerber/Bottom.gbr 	изменено:      kiCAD/SC-STM32L412K8-light_v2/gerber/MaskBottom.gbr 	изменено:      kiCAD/SC-STM32L412K8-light_v2/gerber/MaskTop.gbr 	изменено:      kiCAD/SC-STM32L412K8-light_v2/gerber/NCData.drl 	изменено:      kiCAD/SC-STM32L412K8-light_v2/gerber/SC-STM32L412K8-job.gbrjob 	изменено:      kiCAD/SC-STM32L412K8-light_v2/gerber/SC-STM32L412K8.zip 	изменено:      kiCAD/SC-STM32L412K8-light_v2/gerber/Top.gbr
Parts:
- J13: footprint My-library:SMD-CONN -> lib:conn_mini
- moved J13 11.3 mm to (30.1, 65.1)
- moved J10 0.85 mm to (54.8, 64.2)
- moved BZ1 0.69 mm to (35.3, 64.5)
- moved R15 0.59 mm to (44.3, 65.7)
- moved J15 0.35 mm to (42.0, 66.3)
- moved L1 0.20 mm to (34.0, 55.0)
Routing:
- net Net-(C18-Pad2): track 15.6 -> 11.4 mm
- net Buzer: track 3.45 -> 2.37 mm
- net Net-(C13-Pad1): track 14.5 -> 13.6 mm
- net +BATT: track 65.6 -> 64.7 mm
