File: kiCAD/EQR15_11-6060-PS/EQR15_11-6060-PS.kicad_sch (KiCad schematic)
At the start: 17 parts, among them J1 Conn, J2 Conn, J3 Conn, J4 Conn, J5 Conn

Commit message: новый файл:    Documents/DoZer-current.png 	новый файл:    Documents/LT8410-current.png 	изменено:      kiCAD/EQR15_11-6060-PS/EQR15_11-6060-PS.kicad_pcb 	изменено:      kiCAD/EQR15_11-6060-PS/EQR15_11-6060-PS.kicad_sch
Parts:
- C3: value 10u -> .1
Changed lines of the file:
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@@
       (effects (font (size 1.27 1.27)) (justify left))
     )
-    (property "Value" "10u" (id 1) (at 187.325 84.455 0)
+    (property "Value" ".1" (id 1) (at 187.325 84.455 0)
       (effects (font (size 1.27 1.27)) (justify left))
     )
@@
     )
     (path "/9f4ad8a6-a390-4e8a-9ab7-c3c65e61ff5e"
-      (reference "C3") (unit 1) (value "10u") (footprint "Capacitor_SMD:C_0402_1005Metric")
+      (reference "C3") (unit 1) (value ".1") (footprint "Capacitor_SMD:C_0402_1005Metric")
     )
     (path "/48cc1b0e-2414-4ac6-840b-68be1b3a53dc"
