File: kiCAD/ERQ15_11-6060-SiPM/ERQ15_11-6060-SiPM.kicad_pcb (KiCad board)
At the start: 2 copper layers, 14 x 14 mm, 16 parts, among them J1 Conn, J2 Conn, J3 Conn, J4 Conn, U1 MCP1700x-280xxTT

Commit message: изменено:      kiCAD/ERQ15_11-6060-SiPM/ERQ15_11-6060-SiPM.kicad_pcb 	изменено:      kiCAD/ERQ15_11-6060-SiPM/ERQ15_11-6060-SiPM.kicad_prl 	изменено:      kiCAD/ERQ15_11-6060-SiPM/ERQ15_11-6060-SiPM.kicad_pro 	изменено:      kiCAD/ERQ15_11-6060-SiPM/ERQ15_11-6060-SiPM.kicad_sch 	изменено:      kiCAD/ERQ15_11-6060-SiPM/fp-info-cache
Parts:
- removed D2: OPA835, Package_TO_SOT_SMD:SOT-23-6
- removed R6: 1k, Resistor_SMD:R_0402_1005Metric
- added C2: 10u, Capacitor_SMD:C_1206_3216Metric, B.Cu at (90.9, 60.9)
- added U2: OPA354, Package_TO_SOT_SMD:SOT-23-5, B.Cu at (95.4, 61.0)
- C4: value 10n -> 2p
- moved J4 53.8 mm to (98.9, 60.4)
- moved R5 48.0 mm to (97.0, 59.0)
- moved C3 46.9 mm to (92.8, 60.5)
- moved R7 46.9 mm to (96.6, 63.2)
- moved D1 46.9 mm to (95.0, 60.4)
- moved J1 46.9 mm to (91.9, 63.7)
- moved R1 46.9 mm to (98.1, 62.5)
- moved R2 46.9 mm to (94.3, 63.2)
- moved J2 46.8 mm to (96.8, 56.6)
- moved U1 46.6 mm to (92.8, 57.8)
- moved J3 46.2 mm to (98.7, 59.0)
- moved C4 45.7 mm to (97.0, 58.0)
- moved L1 45.6 mm to (95.3, 57.0), turned to -90 degrees
- moved C1 44.8 mm to (93.6, 55.8)
Connections:
- C4 pad 1: Net-(C4-Pad1) -> Net-(U2--)
- R2 pad 2: Net-(D2-Pad4) -> Net-(U2--)
- R5 pad 1: Net-(C4-Pad1) -> Net-(C4-Pad2)
- R5 pad 2: Net-(D2-Pad4) -> Net-(U2--)
Routing:
- net Net-(U2--): track 0.00 -> 7.31 mm
- net Net-(D2-Pad4): track 5.84 -> 0.00 mm
- net Net-(C4-Pad1): track 2.33 -> 0.00 mm
- net Net-(D1-C): track 1.85 -> 3.56 mm
- net Net-(C4-Pad2): track 2.10 -> 3.74 mm
- net +3V0: track 3.79 -> 2.49 mm
- net GND: track 15.6 -> 14.4 mm
- net Net-(C1-Pad2): track 2.12 -> 2.93 mm
- net (no net): vias 0 -> 6
